Commit message: Dodalem pliki pozwalajace na odpalenie modelu w Rviz i gazebo

File: simulation/ros2_ws/src/hexapod/hexapod_description/urdf/platform/platform.xacro (robot description, xacro)
@@ -32,4 +32,9 @@
       </inertial>
     </link>
+    <!-- <joint name="base_to_world" type="fixed">
+      <parent link="world"/>
+      <child link="base_link"/>
+      <origin xyz="0 0 0" rpy="0 0 0"/>
+    </joint> -->
     <gazebo reference="base_link">
       <visual>

Commit message: Mozna odpalic ros2 launch hexapod_moveit_config demo.launch.py i ustawic jakis ruch w Rviz

File: simulation/ros2_ws/src/hexapod/hexapod_description/urdf/platform/platform.xacro (robot description, xacro)
@@ -13,7 +13,7 @@
         </geometry>
         <material name="green">
-          <color rgba="0 1 0 1"/>
+          <color rgba="0.0 1.0 0.0 1.0"/>
         </material>
-        <origin xyz="0 0 0" rpy="0 0 0"/>
+        <origin xyz="0.0 0.0 0.0" rpy="0.0 0.0 0.0"/>
       </visual>
       <collision>
@@ -21,8 +21,8 @@
           <mesh filename="file://$(find hexapod_description)/meshes/platform.stl"/>
         </geometry>
-        <origin xyz="0 0 0" rpy="0 0 0"/>
+        <origin xyz="0.0 0.0 0.0" rpy="0.0 0.0 0.0"/>
       </collision>
       <inertial>
-        <origin xyz="0 0 0" rpy="0 0 0"/>
+        <origin xyz="0.0 0.0 0.0" rpy="0.0 0.0 0.0"/>
         <mass value="${base_mass}"/>
         <inertia
@@ -40,7 +40,7 @@
       <visual>
         <material>
-          <ambient>0 0.7 0 1</ambient>
-          <diffuse>0 0.7 0 1</diffuse>
-          <specular>0 0.7 0 1</specular>
+          <ambient>0.0 0.7 0.0 1.0</ambient>
+          <diffuse>0.0 0.7 0.0 1.0</diffuse>
+          <specular>0.0 0.7 0.0 1.0</specular>
         </material>
       </visual>

File: simulation/ros2_ws/src/hexapod/hexapod_description/urdf/up_section/up_section.xacro (robot description, xacro)
@@ -1,8 +1,8 @@
 <?xml version="1.0"?>
 <robot xmlns:xacro="http://www.ros.org/wiki/xacro">
-  <xacro:property name="wheel_mass" value="1" />
-  <xacro:property name="ixx" value="1" />
-  <xacro:property name="iyy" value="1" />
-  <xacro:property name="izz" value="1" />
+  <xacro:property name="wheel_mass" value="1.0" />
+  <xacro:property name="ixx" value="1.0" />
+  <xacro:property name="iyy" value="1.0" />
+  <xacro:property name="izz" value="1.0" />
 <!-- tak można przekazać parametr -->
 <!--  <xacro:macro name="mecanum_wheel" params="prefix side x_reflect y_reflect"> -->
@@ -10,5 +10,5 @@
     <link name="up_section">
       <visual>
-        <origin xyz="0 0 0" rpy="0 0 0"/>
+        <origin xyz="0.0 0.0 0.0" rpy="0.0 0.0 0.0"/>
         <geometry>
           <mesh filename="file://$(find hexapod_description)/meshes/leg_up.stl"/>
@@ -19,5 +19,5 @@
       </visual>
       <collision>
-        <origin xyz="0 0 0" rpy="0 0 0"/>
+        <origin xyz="0.0 0.0 0.0" rpy="0.0 0.0 0.0"/>
         <geometry>
           <mesh filename="file://$(find hexapod_description)/meshes/leg_up.stl"/>
@@ -25,17 +25,17 @@
       </collision>
       <inertial>
-        <origin xyz="0 0 0" rpy="0 0 0"/>
+        <origin xyz="0.0 0.0 0.0" rpy="0.0 0.0 0.0"/>
         <mass value="${wheel_mass}"/>
         <inertia
-          ixx="${ixx}" ixy="0" ixz="0"
-          iyy="${iyy}" iyz="0"
+          ixx="${ixx}" ixy="0.0" ixz="0.0"
+          iyy="${iyy}" iyz="0.0"
           izz="${izz}"/>
       </inertial>
     </link>
     <joint name="up_section_joint" type="revolute">
-      <axis xyz="0 0 1"/>
+      <axis xyz="0.0 0.0 1.0"/>
       <parent link="base_link"/>
       <child link="up_section"/>
-      <origin xyz="-0.0052386 0.097578 0.0015" rpy="0 0 0"/>
+      <origin xyz="-0.0052386 0.097578 0.0015" rpy="0.0 0.0 0.0"/>
       <!-- ograniczenie kątów -30 do 30 stopni -->
       <limit effort="5.0" velocity="1.0" lower="-0.5236" upper="0.5236"/>
