Commit message: prawdiłowe linki i jointy jednej nogi

File: simulation/ros2_ws/src/hexapod/hexapod_description/urdf/down_section/down_section.xacro (robot description, xacro)
@@ -10,5 +10,5 @@
     <link name="down_section">
       <visual>
-        <origin xyz="0.0 0.0 0.0" rpy="0.0 0.0 0.0"/>
+        <origin xyz="0.0  0.055874  -0.0577" rpy="0.0 0.0 0.0"/>
         <geometry>
           <mesh filename="file://$(find hexapod_description)/meshes/leg_down.stl"/>
@@ -19,5 +19,5 @@
       </visual>
       <collision>
-        <origin xyz="0.0 0.0 0.0" rpy="0.0 0.0 0.0"/>
+        <origin xyz="0.        0.0  0.0" rpy="0.0 0.0 0.0"/>
         <geometry>
           <mesh filename="file://$(find hexapod_description)/meshes/leg_down.stl"/>
@@ -25,5 +25,5 @@
       </collision>
       <inertial>
-        <origin xyz="0.0 0.0 0.0" rpy="0.0 0.0 0.0"/>
+        <origin xyz="0.0        0.0 0.0" rpy="0.0 0.0 0.0"/>
         <mass value="${wheel_mass}"/>
         <inertia
@@ -34,8 +34,8 @@
     </link>
     <joint name="down_section_joint" type="revolute">
-      <axis xyz="0.0 0.0 1.0"/>
-      <parent link="base_link"/>
+      <axis xyz="1.0 0.0 0.0"/>
+      <parent link="mid_section"/>
       <child link="down_section"/>
-      <origin xyz="0.01148 0.14978 -0.001242" rpy="0.0 0.0 0.0"/>
+      <origin xyz="0.0        0.09  0.005618" rpy="0.0 0.0 0.0"/>
       <!-- ograniczenie kątów -30 do 30 stopni -->
       <limit effort="5.0" velocity="1.0" lower="-0.5236" upper="0.5236"/>

File: simulation/ros2_ws/src/hexapod/hexapod_description/urdf/middle_section/middle_section.xacro (robot description, xacro)
@@ -10,5 +10,5 @@
     <link name="mid_section">
       <visual>
-        <origin xyz="0.0 0.0 0.0" rpy="0.0 0.0 0.0"/>
+        <origin xyz="0.0 0.03637 0.00361" rpy="0.0 0.0 0.0"/>
         <geometry>
           <mesh filename="file://$(find hexapod_description)/meshes/leg_mid.stl"/>
@@ -33,19 +33,9 @@
       </inertial>
     </link>
-<!-- joint do górnej -->
     <joint name="mid_section_joint_1" type="revolute">
       <axis xyz="1.0 0.0 0.0"/>
       <parent link="up_section"/>
       <child link="mid_section"/>
-      <origin xyz="0.007288 0.031914 0.00522" rpy="0.0 0.0 0.0"/>
-      <!-- ograniczenie kątów -30 do 30 stopni -->
-      <limit effort="5.0" velocity="1.0" lower="-0.5236" upper="0.5236"/>
-    </joint>
-<!-- joint do dolnej -->
-    <joint name="mid_section_joint_2" type="revolute">
-      <axis xyz="1.0 0.0 0.0"/>
-      <parent link="up_section"/>
-      <child link="mid_section"/>
-      <origin xyz="0.007288 0.031914 0.00522" rpy="0.0 0.0 0.0"/>
+      <origin xyz="0.0       0.03062  -0.01454" rpy="0.0 0.0 0.0"/>
       <!-- ograniczenie kątów -30 do 30 stopni -->
       <limit effort="5.0" velocity="1.0" lower="-0.5236" upper="0.5236"/>

File: simulation/ros2_ws/src/hexapod/hexapod_description/urdf/up_section/up_section.xacro (robot description, xacro)
@@ -33,9 +33,9 @@
       </inertial>
     </link>
-    <joint name="up_section_joint" type="revolute">
+    <joint name="up_section_joint_1" type="revolute">
       <axis xyz="0.0 0.0 1.0"/>
       <parent link="base_link"/>
       <child link="up_section"/>
-      <origin xyz="-0.0052386 0.097578 0.0015" rpy="0.0 0.0 0.0"/>
+      <origin xyz="0.0  0.069   0.000952" rpy="0.0 0.0 0.0"/>
       <!-- ograniczenie kątów -30 do 30 stopni -->
       <limit effort="5.0" velocity="1.0" lower="-0.5236" upper="0.5236"/>
