Commit message: added inertia
TODO: update legs data after we move to new hexapod model, now length/radiu etc are from old model

File: simulation/ros2_ws_hex/src/open_manipulator_description/urdf/om_x/open_manipulator_x_arm.urdf.xacro (robot description, xacro)
@@ -3,7 +3,48 @@
   <xacro:property name="base_mass" value="4.6" />
   <xacro:property name="wheel_mass" value="1.0" />
+  <!-- Define global properties -->
+  <xacro:property name="base_radius" value="0.15"/>
+  <xacro:property name="base_height" value="0.02"/>
+  <xacro:property name="leg_length_upper" value="0.03"/>
+  <xacro:property name="leg_length_middle" value="0.089"/>
+  <xacro:property name="leg_length_lower" value="0.164"/>
+  <xacro:property name="leg_radius" value="0.02"/>
+  <xacro:property name="PI_const" value="3.1415926"/>
+  <xacro:property name="mass_upper" value="0.1" />
+  <xacro:property name="mass_middle" value="0.1" />
+  <xacro:property name="mass_lower" value="0.1" />
+  <xacro:property name="dx_upp" value="${leg_radius * 2}"/>
+  <xacro:property name="dy_upp" value="${leg_radius * 2}"/>
+  <xacro:property name="dz_upp" value="${leg_length_upper}"/>
+  <xacro:property name="dx_mid" value="${leg_radius * 2}"/>
+  <xacro:property name="dy_mid" value="${leg_radius * 2}"/>
+  <xacro:property name="dz_mid" value="${leg_length_middle}"/>
+  <xacro:property name="dx_low" value="${leg_radius * 2}"/>
+  <xacro:property name="dy_low" value="${leg_radius * 2}"/>
+  <xacro:property name="dz_low" value="${leg_length_lower}"/>
   <xacro:property name="ixx" value="1.0"/>
   <xacro:property name="iyy" value="1.0"/>
   <xacro:property name="izz" value="1.0"/>
+  <!--upper leg -->
+  <xacro:property name="ixx_upp" value="${dy_upp*dy_upp + dz_upp*dz_upp}"/>
+  <xacro:property name="iyy_upp" value="${dx_upp*dx_upp + dz_upp*dz_upp}"/>
+  <xacro:property name="izz_upp" value="${dx_upp*dx_upp + dy_upp*dy_upp}"/>
+  <xacro:property name="ixy_upp" value="(-dx_upp * dy_upp)"/>
+  <xacro:property name="ixz_upp" value="(-dx_upp * dz_upp)"/>
+  <xacro:property name="iyz_upp" value="(-dy_upp * dz_upp)"/>
+  <!--middle leg -->
+  <xacro:property name="ixx_mid" value="${dy_mid*dy_mid + dz_mid*dz_mid}"/>
+  <xacro:property name="iyy_mid" value="${dx_mid*dx_mid + dz_mid*dz_mid}"/>
+  <xacro:property name="izz_mid" value="${dx_mid*dx_mid + dy_mid*dy_mid}"/>
+  <xacro:property name="ixy_mid" value="(-dx_mid * dy_mid)"/>
+  <xacro:property name="ixz_mid" value="(-dx_mid * dz_mid)"/>
+  <xacro:property name="iyz_mid" value="(-dy_mid * dz_mid)"/>
+  <!-- lower leg -->
+  <xacro:property name="ixx_low" value="${dy_low*dy_low + dz_low*dz_low}"/>
+  <xacro:property name="iyy_low" value="${dx_low*dx_low + dz_low*dz_low}"/>
+  <xacro:property name="izz_low" value="${dx_low*dx_low + dy_low*dy_low}"/>
+  <xacro:property name="ixy_low" value="(-dx_low * dy_low)"/>
+  <xacro:property name="ixz_low" value="(-dx_low * dz_low)"/>
+  <xacro:property name="iyz_low" value="(-dy_low * dz_low)"/>
   <xacro:macro name="open_manipulator_x" params="prefix=''">
     <xacro:property
@@ -66,7 +107,7 @@
         <mass value="${wheel_mass}"/>
         <inertia
-          ixx="${ixx}" ixy="0.0" ixz="0.0"
-          iyy="${iyy}" iyz="0.0"
-          izz="${izz}"/>
+          ixx="${ixx_upp}" ixy="${ixy_upp}" ixz="${ixz_upp}"
+          iyy="${iyy_upp}" iyz="${iyz_upp}"
+          izz="${izz_upp}"/>
       </inertial>
     </link>
@@ -101,7 +142,7 @@
         <mass value="${wheel_mass}"/>
         <inertia
-          ixx="${ixx}" ixy="0.0" ixz="0.0"
-          iyy="${iyy}" iyz="0.0"
-          izz="${izz}"/>
+          ixx="${ixx_mid}" ixy="${ixy_mid}" ixz="${ixz_mid}"
+          iyy="${iyy_mid}" iyz="${iyz_mid}"
+          izz="${izz_mid}"/>
       </inertial>
     </link>
@@ -136,7 +177,7 @@
         <mass value="${wheel_mass}"/>
         <inertia
-          ixx="${ixx}" ixy="0.0" ixz="0.0"
-          iyy="${iyy}" iyz="0.0"
-          izz="${izz}"/>
+          ixx="${ixx_low}" ixy="${ixy_low}" ixz="${ixz_low}"
+          iyy="${iyy_low}" iyz="${iyz_low}"
+          izz="${izz_low}"/>
       </inertial>
     </link>

Commit message: wstawione prawidlowe modele nogi 5 i poprawione linki i jointy nogi 5

File: simulation/ros2_ws_hex/src/open_manipulator_description/urdf/om_x/open_manipulator_x_arm.urdf.xacro (robot description, xacro)
@@ -13,5 +13,5 @@
      <link name="${prefix}link1">
        <visual>
-         <origin xyz="0 0 0" rpy="0 0 0"/>
+         <origin xyz="-0.001140 0.000016 -0.002812" rpy="0 0 0"/>
          <geometry>
            <mesh filename="${meshes_file_direction}/platform.stl" scale="1.0 1.0 1.0"/>
@@ -40,5 +40,5 @@
        <parent link="${prefix}link1"/>
        <child link="${prefix}link2"/>
-       <origin xyz="0.0  0.067311   0.0" rpy="0 0 0"/>
+       <origin xyz="-0.00431  -0.097816   0.00596" rpy="0 0 0"/>
        <axis xyz="0.0 0.0 1.0"/>
        <limit effort="5.0" velocity="1.0" lower="-0.5236" upper="0.5236"/>
@@ -48,5 +48,5 @@
      <link name="${prefix}link2">
        <visual>
-         <origin xyz="0	0.001689	0.000952" rpy="0 0 0"/>
+         <origin xyz="0.000493	-0.021762	-0.000419" rpy="0 0 0"/>
          <geometry>
            <mesh filename="${meshes_file_direction}/leg_up.stl" scale="1.0 1.0 1.0"/>
@@ -75,5 +75,5 @@
        <parent link="${prefix}link2"/>
        <child link="${prefix}link3"/>
-       <origin xyz="0	0.02984	-0.012092" rpy="0 0 0"/>
+       <origin xyz="0.0	-0.031057	-0.020002" rpy="0 0 0"/>
        <axis xyz="1 0 0"/>
        <limit effort="5.0" velocity="1.0" lower="-0.5236" upper="0.5236"/>
@@ -83,5 +83,5 @@
      <link name="${prefix}link3">
        <visual>
-         <origin xyz="0	0.038839	0.002114" rpy="0 0 0"/>
+         <origin xyz="0.0	-0.041	0.000546" rpy="0 0 0"/>
          <geometry>
            <mesh filename="${meshes_file_direction}/leg_mid.stl" scale="1.0 1.0 1.0"/>
@@ -110,5 +110,5 @@
        <parent link="${prefix}link3"/>
        <child link="${prefix}link4"/>
-       <origin xyz="0	0.089024	0.005843" rpy="0 0 0"/>
+       <origin xyz="0.0	-0.089946	0.00505" rpy="0 0 0"/>
        <axis xyz="1 0 0"/>
        <limit effort="5.0" velocity="1.0" lower="-0.5236" upper="0.5236"/>
@@ -118,5 +118,5 @@
      <link name="${prefix}link4">
        <visual>
-         <origin xyz="0	0.057622	-0.058093" rpy="0 0 0"/>
+         <origin xyz="-0.000265	-0.064842	0.0" rpy="0 0 0"/>
          <geometry>
            <mesh filename="${meshes_file_direction}/leg_down.stl" scale="1.0 1.0 1.0"/>

Commit message: cały model wstawiony do symulacji

File: simulation/ros2_ws_hex/src/open_manipulator_description/urdf/om_x/open_manipulator_x_arm.urdf.xacro (robot description, xacro)
@@ -10,5 +10,5 @@
        name="meshes_file_direction"
        value="package://open_manipulator_description/meshes"/>
- <!-- PLATFORMA -->
+<!-- PLATFORMA -->
      <link name="${prefix}link1">
        <visual>
@@ -36,4 +36,430 @@
        </inertial>
      </link>
+  <!-- LEG 1!!!!!!!!!!!!!!!!!!!!!!!!!!!!!!!!!!!!!!!!!!!!!!!!!!!!!!!!!!!!!!! -->
+     <!-- PLATFORMA - UP_SECTION -->
+     <joint name="${prefix}joint1_1" type="revolute">
+       <parent link="${prefix}link1"/>
+       <child link="${prefix}link2_1"/>
+       <origin xyz="-0.062614  0.067285   0.00596" rpy="0 0 0"/>
+       <axis xyz="0.0 0.0 1.0"/>
+       <limit effort="5.0" velocity="1.0" lower="-0.5236" upper="0.5236"/>
+       <dynamics damping="0.1"/>
+     </joint>
+   <!-- UP_SECTION -->
+     <link name="${prefix}link2_1">
+       <visual>
+         <origin xyz="-0.013611	0.016988 -0.000419" rpy="0 0 0"/>
+         <geometry>
+           <mesh filename="${meshes_file_direction}/1_leg_up.stl" scale="1.0 1.0 1.0"/>
+         </geometry>
+         <material name="grey">
+           <color rgba="0.2 0.2 0.2 1"/>
+         </material>
+       </visual>
+       <collision>
+         <origin xyz="0	0.001689	0.000952" rpy="0 0 0"/>
+         <geometry>
+           <mesh filename="${meshes_file_direction}/1_leg_up.stl" scale="1.0 1.0 1.0"/>
+         </geometry>
+       </collision>
+        <inertial>
+         <origin xyz="0.0 0.0 0.0" rpy="0.0 0.0 0.0"/>
+         <mass value="${wheel_mass}"/>
+         <inertia
+           ixx="${ixx}" ixy="0.0" ixz="0.0"
+           iyy="${iyy}" iyz="0.0"
+           izz="${izz}"/>
+       </inertial>
+     </link>
+   <!-- UP_SECTION - MID_SECTION -->
+     <joint name="${prefix}joint2_1" type="revolute">
+       <parent link="${prefix}link2_1"/>
+       <child link="${prefix}link3_1"/>
+       <origin xyz="-0.018864	0.024671	-0.020002" rpy="0 0 0"/>
+       <axis xyz="0.6074290528 0.794374 0"/>
+       <limit effort="5.0" velocity="1.0" lower="-0.5236" upper="0.5236"/>
+       <dynamics damping="0.1"/>
+     </joint>
+   <!-- MID_SECTION -->
+     <link name="${prefix}link3_1">
+       <visual>
+         <origin xyz="-0.024936	0.032658	0.000547" rpy="0 0 0"/>
+         <geometry>
+           <mesh filename="${meshes_file_direction}/1_leg_mid.stl" scale="1.0 1.0 1.0"/>
+         </geometry>
+         <material name="grey">
+           <color rgba="0.2 0.2 0.2 1"/>
+         </material>
+       </visual>
+       <collision>
+         <origin xyz="0	0.038839	0.002114" rpy="0 0 0"/>
+         <geometry>
+           <mesh filename="${meshes_file_direction}/1_leg_mid.stl" scale="1.0 1.0 1.0"/>
+         </geometry>
+       </collision>
+        <inertial>
+         <origin xyz="0.0 0.0 0.0" rpy="0.0 0.0 0.0"/>
+         <mass value="${wheel_mass}"/>
+         <inertia
+           ixx="${ixx}" ixy="0.0" ixz="0.0"
+           iyy="${iyy}" iyz="0.0"
+           izz="${izz}"/>
+       </inertial>
+     </link>
+   <!-- MID_SECTION - DOWN_SECTION -->
+     <joint name="${prefix}joint3_1" type="revolute">
+       <parent link="${prefix}link3_1"/>
+       <child link="${prefix}link4_1"/>
+       <origin xyz="-0.054636	0.071451	0.00505" rpy="0 0 0"/>
+       <axis xyz="0.6074290528 0.794374 0"/>
+       <limit effort="5.0" velocity="1.0" lower="-0.5236" upper="0.5236"/>
+       <dynamics damping="0.1"/>
+     </joint>
+   <!-- DOWN_SECTION -->
+     <link name="${prefix}link4_1">
+       <visual>
+         <origin xyz="-0.039176	0.05167	0" rpy="0 0 0"/>
+         <geometry>
+           <mesh filename="${meshes_file_direction}/1_leg_down.stl" scale="1.0 1.0 1.0"/>
+         </geometry>
+         <material name="grey">
+           <color rgba="0.2 0.2 0.2 1"/>
+         </material>
+       </visual>
+       <collision>
+         <origin xyz="0	0.057622	-0.058093" rpy="0 0 0"/>
+         <geometry>
+           <mesh filename="${meshes_file_direction}/1_leg_down.stl" scale="1.0 1.0 1.0"/>
+         </geometry>
+       </collision>
+        <inertial>
+         <origin xyz="0.0        0.0 0.0" rpy="0.0 0.0 0.0"/>
+         <mass value="${wheel_mass}"/>
+         <inertia
+           ixx="${ixx}" ixy="0.0" ixz="0.0"
+           iyy="${iyy}" iyz="0.0"
+           izz="${izz}"/>
+       </inertial>
+     </link>
+     <!-- LEG 2!!!!!!!!!!!!!!!!!!!!!!!!!!!!!!!!!!!!!!!!!!!!!!!!!!!!!!!!!!!!!!!!!!!!!!!1 -->
+     <!-- PLATFORMA - UP_SECTION -->
+     <!-- PLATFORMA - UP_SECTION -->
+     <joint name="${prefix}joint1_2" type="revolute">
+       <parent link="${prefix}link1"/>
+       <child link="${prefix}link2_2"/>
+       <origin xyz="-0.00431  0.097816   0.00596" rpy="0 0 0"/>
+       <axis xyz="0.0 0.0 1.0"/>
+       <limit effort="5.0" velocity="1.0" lower="-0.5236" upper="0.5236"/>
+       <dynamics damping="0.1"/>
+     </joint>
+   <!-- UP_SECTION -->
+     <link name="${prefix}link2_2">
+       <visual>
+         <origin xyz="-0.000493	0.021762	-0.000419" rpy="0 0 0"/>
+         <geometry>
+           <mesh filename="${meshes_file_direction}/2_leg_up.stl" scale="1.0 1.0 1.0"/>
+         </geometry>
+         <material name="grey">
+           <color rgba="0.2 0.2 0.2 1"/>
+         </material>
+       </visual>
+       <collision>
+         <origin xyz="0	0.001689	0.000952" rpy="0 0 0"/>
+         <geometry>
+           <mesh filename="${meshes_file_direction}/2_leg_up.stl" scale="1.0 1.0 1.0"/>
+         </geometry>
+       </collision>
+        <inertial>
+         <origin xyz="0.0 0.0 0.0" rpy="0.0 0.0 0.0"/>
+         <mass value="${wheel_mass}"/>
+         <inertia
+           ixx="${ixx}" ixy="0.0" ixz="0.0"
+           iyy="${iyy}" iyz="0.0"
+           izz="${izz}"/>
+       </inertial>
+     </link>
+   <!-- UP_SECTION - MID_SECTION -->
+     <joint name="${prefix}joint2_2" type="revolute">
+       <parent link="${prefix}link2_2"/>
+       <child link="${prefix}link3_2"/>
+       <origin xyz="0.0	0.031057	-0.020002" rpy="0 0 0"/>
+       <axis xyz="-1 0 0"/>
+       <limit effort="5.0" velocity="1.0" lower="-0.5236" upper="0.5236"/>
+       <dynamics damping="0.1"/>
+     </joint>
+   <!-- MID_SECTION -->
+     <link name="${prefix}link3_2">
+       <visual>
+         <origin xyz="0.0	0.041	0.000546" rpy="0 0 0"/>
+         <geometry>
+           <mesh filename="${meshes_file_direction}/2_leg_mid.stl" scale="1.0 1.0 1.0"/>
+         </geometry>
+         <material name="grey">
+           <color rgba="0.2 0.2 0.2 1"/>
+         </material>
+       </visual>
+       <collision>
+         <origin xyz="0	0.038839	0.002114" rpy="0 0 0"/>
+         <geometry>
+           <mesh filename="${meshes_file_direction}/2_leg_mid.stl" scale="1.0 1.0 1.0"/>
+         </geometry>
+       </collision>
+        <inertial>
+         <origin xyz="0.0 0.0 0.0" rpy="0.0 0.0 0.0"/>
+         <mass value="${wheel_mass}"/>
+         <inertia
+           ixx="${ixx}" ixy="0.0" ixz="0.0"
+           iyy="${iyy}" iyz="0.0"
+           izz="${izz}"/>
+       </inertial>
+     </link>
+   <!-- MID_SECTION - DOWN_SECTION -->
+     <joint name="${prefix}joint3_2" type="revolute">
+       <parent link="${prefix}link3_2"/>
+       <child link="${prefix}link4_2"/>
+       <origin xyz="0.0	0.089946	0.00505" rpy="0 0 0"/>
+       <axis xyz="-1 0 0"/>
+       <limit effort="5.0" velocity="1.0" lower="-0.5236" upper="0.5236"/>
+       <dynamics damping="0.1"/>
+     </joint>
+   <!-- DOWN_SECTION -->
+     <link name="${prefix}link4_2">
+       <visual>
+         <origin xyz="0.000265	0.064842	0.0" rpy="0 0 0"/>
+         <geometry>
+           <mesh filename="${meshes_file_direction}/2_leg_down.stl" scale="1.0 1.0 1.0"/>
+         </geometry>
+         <material name="grey">
+           <color rgba="0.2 0.2 0.2 1"/>
+         </material>
+       </visual>
+       <collision>
+         <origin xyz="0	0.057622	-0.058093" rpy="0 0 0"/>
+         <geometry>
+           <mesh filename="${meshes_file_direction}/2_leg_down.stl" scale="1.0 1.0 1.0"/>
+         </geometry>
+       </collision>
+        <inertial>
+         <origin xyz="0.0        0.0 0.0" rpy="0.0 0.0 0.0"/>
+         <mass value="${wheel_mass}"/>
+         <inertia
+           ixx="${ixx}" ixy="0.0" ixz="0.0"
+           iyy="${iyy}" iyz="0.0"
+           izz="${izz}"/>
+       </inertial>
+     </link>
+  <!-- LEG 3!!!!!!!!!!!!!!!!!!!!!!!!!!!!!!!!!!!!!!!!!!!!!!!!!!!!!!!!!!!!!!! -->
+     <!-- PLATFORMA - UP_SECTION -->
+     <joint name="${prefix}joint1_3" type="revolute">
+       <parent link="${prefix}link1"/>
+       <child link="${prefix}link2_3"/>
+       <origin xyz="0.056235  0.073938   0.00596" rpy="0 0 0"/>
+       <axis xyz="0.0 0.0 1.0"/>
+       <limit effort="5.0" velocity="1.0" lower="-0.5236" upper="0.5236"/>
+       <dynamics damping="0.1"/>
+     </joint>
+   <!-- UP_SECTION -->
+     <link name="${prefix}link2_3">
+       <visual>
+         <origin xyz="0.012827	0.017587 -0.000419" rpy="0 0 0"/>
+         <geometry>
+           <mesh filename="${meshes_file_direction}/3_leg_up.stl" scale="1.0 1.0 1.0"/>
+         </geometry>
+         <material name="grey">
+           <color rgba="0.2 0.2 0.2 1"/>
+         </material>
+       </visual>
+       <collision>
+         <origin xyz="0	0.001689	0.000952" rpy="0 0 0"/>
+         <geometry>
+           <mesh filename="${meshes_file_direction}/3_leg_up.stl" scale="1.0 1.0 1.0"/>
+         </geometry>
+       </collision>
+        <inertial>
+         <origin xyz="0.0 0.0 0.0" rpy="0.0 0.0 0.0"/>
+         <mass value="${wheel_mass}"/>
+         <inertia
+           ixx="${ixx}" ixy="0.0" ixz="0.0"
+           iyy="${iyy}" iyz="0.0"
+           izz="${izz}"/>
+       </inertial>
+     </link>
+   <!-- UP_SECTION - MID_SECTION -->
+     <joint name="${prefix}joint2_3" type="revolute">
+       <parent link="${prefix}link2_3"/>
+       <child link="${prefix}link3_3"/>
+       <origin xyz="0.018864	0.024671	-0.020002" rpy="0 0 0"/>
+       <axis xyz="-0.794374 0.6074290528 0"/>
+       <limit effort="5.0" velocity="1.0" lower="-0.5236" upper="0.5236"/>
+       <dynamics damping="0.1"/>
+     </joint>
+   <!-- MID_SECTION -->
+     <link name="${prefix}link3_3">
+       <visual>
+         <origin xyz="0.024936	0.032658	0.000547" rpy="0 0 0"/>
+         <geometry>
+           <mesh filename="${meshes_file_direction}/3_leg_mid.stl" scale="1.0 1.0 1.0"/>
+         </geometry>
+         <material name="grey">
+           <color rgba="0.2 0.2 0.2 1"/>
+         </material>
+       </visual>
+       <collision>
+         <origin xyz="0	0.038839	0.002114" rpy="0 0 0"/>
+         <geometry>
+           <mesh filename="${meshes_file_direction}/3_leg_mid.stl" scale="1.0 1.0 1.0"/>
+         </geometry>
+       </collision>
+        <inertial>
+         <origin xyz="0.0 0.0 0.0" rpy="0.0 0.0 0.0"/>
+         <mass value="${wheel_mass}"/>
+         <inertia
+           ixx="${ixx}" ixy="0.0" ixz="0.0"
+           iyy="${iyy}" iyz="0.0"
+           izz="${izz}"/>
+       </inertial>
+     </link>
+   <!-- MID_SECTION - DOWN_SECTION -->
+     <joint name="${prefix}joint3_3" type="revolute">
+       <parent link="${prefix}link3_3"/>
+       <child link="${prefix}link4_3"/>
+       <origin xyz="0.054636	0.071451	0.00505" rpy="0 0 0"/>
+       <axis xyz="-0.794374 0.6074290528 0"/>
+       <limit effort="5.0" velocity="1.0" lower="-0.5236" upper="0.5236"/>
+       <dynamics damping="0.1"/>
+     </joint>
+   <!-- DOWN_SECTION -->
+     <link name="${prefix}link4_3">
+       <visual>
+         <origin xyz="0.039176	0.05167	0" rpy="0 0 0"/>
+         <geometry>
+           <mesh filename="${meshes_file_direction}/3_leg_down.stl" scale="1.0 1.0 1.0"/>
+         </geometry>
+         <material name="grey">
+           <color rgba="0.2 0.2 0.2 1"/>
+         </material>
+       </visual>
+       <collision>
+         <origin xyz="0	0.057622	-0.058093" rpy="0 0 0"/>
+         <geometry>
+           <mesh filename="${meshes_file_direction}/3_leg_down.stl" scale="1.0 1.0 1.0"/>
+         </geometry>
+       </collision>
+        <inertial>
+         <origin xyz="0.0        0.0 0.0" rpy="0.0 0.0 0.0"/>
+         <mass value="${wheel_mass}"/>
+         <inertia
+           ixx="${ixx}" ixy="0.0" ixz="0.0"
+           iyy="${iyy}" iyz="0.0"
+           izz="${izz}"/>
+       </inertial>
+     </link>
+  <!-- LEG 4!!!!!!!!!!!!!!!!!!!!!!!!!!!!!!!!!!!!!!!!!!!!!!!!!!!!!!!!!!!!!!! -->
+     <!-- PLATFORMA - UP_SECTION -->
+     <joint name="${prefix}joint1_4" type="revolute">
+       <parent link="${prefix}link1"/>
+       <child link="${prefix}link2_4"/>
+       <origin xyz="0.056235  -0.073938   0.00596" rpy="0 0 0"/>
+       <axis xyz="0.0 0.0 1.0"/>
+       <limit effort="5.0" velocity="1.0" lower="-0.5236" upper="0.5236"/>
+       <dynamics damping="0.1"/>
+     </joint>
+   <!-- UP_SECTION -->
+     <link name="${prefix}link2_4">
+       <visual>
+         <origin xyz="0.013611	-0.016988 -0.000419" rpy="0 0 0"/>
+         <geometry>
+           <mesh filename="${meshes_file_direction}/4_leg_up.stl" scale="1.0 1.0 1.0"/>
+         </geometry>
+         <material name="grey">
+           <color rgba="0.2 0.2 0.2 1"/>
+         </material>
+       </visual>
+       <collision>
+         <origin xyz="0	0.001689	0.000952" rpy="0 0 0"/>
+         <geometry>
+           <mesh filename="${meshes_file_direction}/4_leg_up.stl" scale="1.0 1.0 1.0"/>
+         </geometry>
+       </collision>
+        <inertial>
+         <origin xyz="0.0 0.0 0.0" rpy="0.0 0.0 0.0"/>
+         <mass value="${wheel_mass}"/>
+         <inertia
+           ixx="${ixx}" ixy="0.0" ixz="0.0"
+           iyy="${iyy}" iyz="0.0"
+           izz="${izz}"/>
+       </inertial>
+     </link>
+   <!-- UP_SECTION - MID_SECTION -->
+     <joint name="${prefix}joint2_4" type="revolute">
+       <parent link="${prefix}link2_4"/>
+       <child link="${prefix}link3_4"/>
+       <origin xyz="0.018864	-0.024671	-0.020002" rpy="0 0 0"/>
+       <axis xyz="0.6074290528 0.794374 0"/>
+       <limit effort="5.0" velocity="1.0" lower="-0.5236" upper="0.5236"/>
+       <dynamics damping="0.1"/>
+     </joint>
+   <!-- MID_SECTION -->
+     <link name="${prefix}link3_4">
+       <visual>
+         <origin xyz="0.024936	-0.032658	0.000547" rpy="0 0 0"/>
+         <geometry>
+           <mesh filename="${meshes_file_direction}/4_leg_mid.stl" scale="1.0 1.0 1.0"/>
+         </geometry>
+         <material name="grey">
+           <color rgba="0.2 0.2 0.2 1"/>
+         </material>
+       </visual>
+       <collision>
+         <origin xyz="0	0.038839	0.002114" rpy="0 0 0"/>
+         <geometry>
+           <mesh filename="${meshes_file_direction}/4_leg_mid.stl" scale="1.0 1.0 1.0"/>
+         </geometry>
+       </collision>
+        <inertial>
+         <origin xyz="0.0 0.0 0.0" rpy="0.0 0.0 0.0"/>
+         <mass value="${wheel_mass}"/>
+         <inertia
+           ixx="${ixx}" ixy="0.0" ixz="0.0"
+           iyy="${iyy}" iyz="0.0"
+           izz="${izz}"/>
+       </inertial>
+     </link>
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