Commit message: dodane modele kolizji

File: simulation/ros2_ws_hex/src/hexapod_description/urdf/hexapod_leg.urdf.xacro (robot description, xacro)
@@ -58,7 +58,7 @@
        </visual>
        <collision>
-         <origin xyz="0	0.001689	0.000952" rpy="0 0 0"/>
-         <geometry>
-           <mesh filename="${meshes_file_direction}/1_leg_up.stl" scale="1.0 1.0 1.0"/>
+         <origin xyz="-0.013611	0.016988 -0.000419" rpy="0 0 0"/>
+         <geometry>
+           <mesh filename="${meshes_file_direction}/hitbox_1_leg_up.stl" scale="1.0 1.0 1.0"/>
          </geometry>
        </collision>
@@ -93,7 +93,7 @@
        </visual>
        <collision>
-         <origin xyz="0	0.038839	0.002114" rpy="0 0 0"/>
-         <geometry>
-           <mesh filename="${meshes_file_direction}/1_leg_mid.stl" scale="1.0 1.0 1.0"/>
+         <origin xyz="-0.024936	0.032658	0.000547" rpy="0 0 0"/>
+         <geometry>
+           <mesh filename="${meshes_file_direction}/hitbox_1_leg_mid.stl" scale="1.0 1.0 1.0"/>
          </geometry>
        </collision>
@@ -128,7 +128,7 @@
        </visual>
        <collision>
-         <origin xyz="0	0.057622	-0.058093" rpy="0 0 0"/>
-         <geometry>
-           <mesh filename="${meshes_file_direction}/1_leg_down.stl" scale="1.0 1.0 1.0"/>
+         <origin xyz="-0.039176	0.05167	0" rpy="0 0 0"/>
+         <geometry>
+           <mesh filename="${meshes_file_direction}/hitbox_1_leg_down.stl" scale="1.0 1.0 1.0"/>
          </geometry>
        </collision>
@@ -165,7 +165,7 @@
        </visual>
        <collision>
-         <origin xyz="0	0.001689	0.000952" rpy="0 0 0"/>
-         <geometry>
-           <mesh filename="${meshes_file_direction}/2_leg_up.stl" scale="1.0 1.0 1.0"/>
+         <origin xyz="-0.000493	0.021762	-0.000419" rpy="0 0 0"/>
+         <geometry>
+           <mesh filename="${meshes_file_direction}/hitbox_2_leg_up.stl" scale="1.0 1.0 1.0"/>
          </geometry>
        </collision>
@@ -200,7 +200,7 @@
        </visual>
        <collision>
-         <origin xyz="0	0.038839	0.002114" rpy="0 0 0"/>
-         <geometry>
-           <mesh filename="${meshes_file_direction}/2_leg_mid.stl" scale="1.0 1.0 1.0"/>
+         <origin xyz="0.0	0.041	0.000546" rpy="0 0 0"/>
+         <geometry>
+           <mesh filename="${meshes_file_direction}/hitbox_2_leg_mid.stl" scale="1.0 1.0 1.0"/>
          </geometry>
        </collision>
@@ -235,7 +235,7 @@
        </visual>
        <collision>
-         <origin xyz="0	0.057622	-0.058093" rpy="0 0 0"/>
-         <geometry>
-           <mesh filename="${meshes_file_direction}/2_leg_down.stl" scale="1.0 1.0 1.0"/>
+         <origin xyz="0.000265	0.064842	0.0" rpy="0 0 0"/>
+         <geometry>
+           <mesh filename="${meshes_file_direction}/hitbox_2_leg_down.stl" scale="1.0 1.0 1.0"/>
          </geometry>
        </collision>
@@ -271,7 +271,7 @@
        </visual>
        <collision>
-         <origin xyz="0	0.001689	0.000952" rpy="0 0 0"/>
-         <geometry>
-           <mesh filename="${meshes_file_direction}/3_leg_up.stl" scale="1.0 1.0 1.0"/>
+         <origin xyz="0.012827	0.017587 -0.000419" rpy="0 0 0"/>
+         <geometry>
+           <mesh filename="${meshes_file_direction}/hitbox_3_leg_up.stl" scale="1.0 1.0 1.0"/>
          </geometry>
        </collision>
@@ -306,7 +306,7 @@
        </visual>
        <collision>
-         <origin xyz="0	0.038839	0.002114" rpy="0 0 0"/>
-         <geometry>
-           <mesh filename="${meshes_file_direction}/3_leg_mid.stl" scale="1.0 1.0 1.0"/>
+         <origin xyz=".024936	0.032658	0.000547" rpy="0 0 0"/>
+         <geometry>
+           <mesh filename="${meshes_file_direction}/hitbox_3_leg_mid.stl" scale="1.0 1.0 1.0"/>
          </geometry>
        </collision>
@@ -341,7 +341,7 @@
        </visual>
        <collision>
-         <origin xyz="0	0.057622	-0.058093" rpy="0 0 0"/>
-         <geometry>
-           <mesh filename="${meshes_file_direction}/3_leg_down.stl" scale="1.0 1.0 1.0"/>
+         <origin xyz="0.039176	0.05167	0" rpy="0 0 0"/>
+         <geometry>
+           <mesh filename="${meshes_file_direction}/hitbox_3_leg_down.stl" scale="1.0 1.0 1.0"/>
          </geometry>
        </collision>
@@ -377,7 +377,7 @@
        </visual>
        <collision>
-         <origin xyz="0	0.001689	0.000952" rpy="0 0 0"/>
-         <geometry>
-           <mesh filename="${meshes_file_direction}/4_leg_up.stl" scale="1.0 1.0 1.0"/>
+         <origin xyz="0.013611	-0.016988 -0.000419" rpy="0 0 0"/>
+         <geometry>
+           <mesh filename="${meshes_file_direction}/hitbox_4_leg_up.stl" scale="1.0 1.0 1.0"/>
          </geometry>
        </collision>
@@ -412,7 +412,7 @@
        </visual>
        <collision>
-         <origin xyz="0	0.038839	0.002114" rpy="0 0 0"/>
-         <geometry>
-           <mesh filename="${meshes_file_direction}/4_leg_mid.stl" scale="1.0 1.0 1.0"/>
+         <origin xyz="0.024936	-0.032658	0.000547" rpy="0 0 0"/>
+         <geometry>
+           <mesh filename="${meshes_file_direction}/hitbox_4_leg_mid.stl" scale="1.0 1.0 1.0"/>
          </geometry>
        </collision>
@@ -447,7 +447,7 @@
        </visual>
        <collision>
-         <origin xyz="0	0.057622	-0.058093" rpy="0 0 0"/>
-         <geometry>
-           <mesh filename="${meshes_file_direction}/4_leg_down.stl" scale="1.0 1.0 1.0"/>
+         <origin xyz="0.039176	-0.05167	0" rpy="0 0 0"/>
+         <geometry>
+           <mesh filename="${meshes_file_direction}/hitbox_4_leg_down.stl" scale="1.0 1.0 1.0"/>
          </geometry>
        </collision>
@@ -483,7 +483,7 @@
        </visual>
        <collision>
-         <origin xyz="0	0.001689	0.000952" rpy="0 0 0"/>
-         <geometry>
-           <mesh filename="${meshes_file_direction}/5_leg_up.stl" scale="1.0 1.0 1.0"/>
+         <origin xyz="0.000493	-0.021762	-0.000419" rpy="0 0 0"/>
+         <geometry>
+           <mesh filename="${meshes_file_direction}/hitbox_5_leg_up.stl" scale="1.0 1.0 1.0"/>
          </geometry>
        </collision>
@@ -518,7 +518,7 @@
        </visual>
        <collision>
-         <origin xyz="0	0.038839	0.002114" rpy="0 0 0"/>
-         <geometry>
-           <mesh filename="${meshes_file_direction}/5_leg_mid.stl" scale="1.0 1.0 1.0"/>
+         <origin xyz="00.0	-0.041	0.000546" rpy="0 0 0"/>
+         <geometry>
+           <mesh filename="${meshes_file_direction}/hitbox_5_leg_mid.stl" scale="1.0 1.0 1.0"/>
          </geometry>
        </collision>
@@ -553,7 +553,7 @@
        </visual>
        <collision>
-         <origin xyz="0	0.057622	-0.058093" rpy="0 0 0"/>
-         <geometry>
-           <mesh filename="${meshes_file_direction}/5_leg_down.stl" scale="1.0 1.0 1.0"/>
+         <origin xyz="-0.000265	-0.064842	0.0" rpy="0 0 0"/>
+         <geometry>
+           <mesh filename="${meshes_file_direction}/hitbox_5_leg_down.stl" scale="1.0 1.0 1.0"/>
          </geometry>
        </collision>
@@ -589,7 +589,7 @@
        </visual>
        <collision>
-         <origin xyz="0	0.001689	0.000952" rpy="0 0 0"/>
-         <geometry>
-           <mesh filename="${meshes_file_direction}/1_leg_up.stl" scale="1.0 1.0 1.0"/>
+         <origin xyz="-0.012827	-0.017588 -0.000419" rpy="0 0 0"/>
+         <geometry>
+           <mesh filename="${meshes_file_direction}/hitbox_6_leg_up.stl" scale="1.0 1.0 1.0"/>
          </geometry>
        </collision>
@@ -624,7 +624,7 @@
        </visual>
        <collision>
-         <origin xyz="0	0.038839	0.002114" rpy="0 0 0"/>
-         <geometry>
-           <mesh filename="${meshes_file_direction}/6_leg_mid.stl" scale="1.0 1.0 1.0"/>
+         <origin xyz="-0.024936	-0.032658	0.000547" rpy="0 0 0"/>
+         <geometry>
+           <mesh filename="${meshes_file_direction}/hitbox_6_leg_mid.stl" scale="1.0 1.0 1.0"/>
          </geometry>
        </collision>
@@ -659,7 +659,7 @@
        </visual>
        <collision>
-         <origin xyz="0	0.057622	-0.058093" rpy="0 0 0"/>
-         <geometry>
-           <mesh filename="${meshes_file_direction}/6_leg_down.stl" scale="1.0 1.0 1.0"/>
+         <origin xyz="-0.039176	-0.05167	0" rpy="0 0 0"/>
+         <geometry>
+           <mesh filename="${meshes_file_direction}/hitbox_6_leg_down.stl" scale="1.0 1.0 1.0"/>
          </geometry>
        </collision>

Commit message: poprawka kątów

File: simulation/ros2_ws_hex/src/hexapod_description/urdf/hexapod_leg.urdf.xacro (robot description, xacro)
@@ -77,5 +77,5 @@
        <child link="${prefix}link3_1"/>
        <origin xyz="-0.018864	0.024671	-0.020002" rpy="0 0 0"/>
-       <axis xyz="-0.6074290528 -0.794374 0"/>
+       <axis xyz="-0.794374 -0.6074290528 0"/>
        <limit effort="5.0" velocity="1.0" lower="-0.261799388" upper="1.308996939"/>
        <dynamics damping="0.1"/>
@@ -112,5 +112,5 @@
        <child link="${prefix}link4_1"/>
        <origin xyz="-0.054636	0.071451	0.00505" rpy="0 0 0"/>
-       <axis xyz="-0.6074290528 -0.794374 0"/>
+       <axis xyz="-0.7968540982 -0.6041717854 0"/>
        <limit effort="5.0" velocity="1.0" lower="0" upper="1.570796327"/>
        <dynamics damping="0.1"/>
@@ -431,5 +431,5 @@
        <child link="${prefix}link4_4"/>
        <origin xyz="0.054636	-0.071451	0.00505" rpy="0 0 0"/>
-       <axis xyz="0.6074290528 0.794374 0"/>
+       <axis xyz="0.794374 0.6074290528 0"/>
        <limit effort="5.0" velocity="1.0" lower="0" upper="1.570796327"/>
        <dynamics damping="0.1"/>
