Commit message: added camera to hexapod
 TODO: change its possition and add image integration

File: simulation/ros2_ws_hex/src/hexapod_description/urdf/hexapod.urdf.xacro (robot description, xacro)
@@ -2,4 +2,10 @@
 <!-- OpenManipulator Chain -->
 <robot name="hexapod" xmlns:xacro="http://ros.org/wiki/xacro">
+  <!-- Includes start -->
+<!--
+  <xacro:include filename="lidar.xacro"/>
+-->
+  <xacro:include filename="camera.xacro"/>
+  <!-- Includes end-->
   <xacro:arg name="prefix" default="" />
   <xacro:arg name="use_sim" default="false" />
@@ -32,3 +38,29 @@
     <child link="$(arg prefix)link1"/>
   </joint> -->
+  <!-- Fake left wheel -->
+  <link name="fake_left_wheel"/>
+  <joint name="fake_left_wheel_joint" type="continuous">
+    <parent link="base_link"/>
+    <child link="fake_left_wheel"/>
+    <origin xyz="0 0.1 0" rpy="0 0 0"/>
+    <axis xyz="0 1 0"/>
+  </joint>
+  <!-- Fake right wheel -->
+  <link name="fake_right_wheel"/>
+  <joint name="fake_right_wheel_joint" type="continuous">
+    <parent link="base_link"/>
+    <child link="fake_right_wheel"/>
+    <origin xyz="0 -0.1 0" rpy="0 0 0"/>
+    <axis xyz="0 1 0"/>
+  </joint>
+  <gazebo reference="fake_left_wheel">
+    <mu1>0</mu1>
+    <mu2>0</mu2>
+    <material>Gazebo/Black</material>
+  </gazebo>
+  <gazebo reference="fake_right_wheel">
+    <mu1>0</mu1>
+    <mu2>0</mu2>
+    <material>Gazebo/Black</material>
+  </gazebo>
 </robot>

Commit message: adding hexapod moving with camera

File: simulation/ros2_ws_hex/src/hexapod_description/urdf/hexapod.urdf.xacro (robot description, xacro)
@@ -30,4 +30,32 @@
     </plugin>
   </gazebo>
+  <!-- Fake left wheel -->
+  <link name="fake_left_wheel">
+    <inertial>
+      <mass value="0.01"/>
+      <origin xyz="0 0 0" rpy="0 0 0"/>
+      <inertia ixx="0.001" ixy="0" ixz="0" iyy="0.001" iyz="0" izz="0.001"/>
+    </inertial>
+  </link>
+  <joint name="fake_left_wheel_joint" type="continuous">
+    <parent link="${prefix}link1"/>
+    <child link="fake_left_wheel"/>
+    <origin xyz="0 0.15 0" rpy="0 0 0"/>
+    <axis xyz="0 1 0"/>
+  </joint>
+  <!-- Fake right wheel -->
+  <link name="fake_right_wheel">
+    <inertial>
+      <mass value="0.01"/>
+      <origin xyz="0 0 0" rpy="0 0 0"/>
+      <inertia ixx="0.001" ixy="0" ixz="0" iyy="0.001" iyz="0" izz="0.001"/>
+    </inertial>
+  </link>
+  <joint name="fake_right_wheel_joint" type="continuous">
+    <parent link="${prefix}link1"/>
+    <child link="fake_right_wheel"/>
+    <origin xyz="0 -0.15 0" rpy="0 0 0"/>
+    <axis xyz="0 1 0"/>
+  </joint>
   <!-- World -->
   <!-- <link name="world"/> -->
@@ -38,29 +66,3 @@
     <child link="$(arg prefix)link1"/>
   </joint> -->
-  <!-- Fake left wheel -->
-  <link name="fake_left_wheel"/>
-  <joint name="fake_left_wheel_joint" type="continuous">
-    <parent link="base_link"/>
-    <child link="fake_left_wheel"/>
-    <origin xyz="0 0.1 0" rpy="0 0 0"/>
-    <axis xyz="0 1 0"/>
-  </joint>
-  <!-- Fake right wheel -->
-  <link name="fake_right_wheel"/>
-  <joint name="fake_right_wheel_joint" type="continuous">
-    <parent link="base_link"/>
-    <child link="fake_right_wheel"/>
-    <origin xyz="0 -0.1 0" rpy="0 0 0"/>
-    <axis xyz="0 1 0"/>
-  </joint>
-  <gazebo reference="fake_left_wheel">
-    <mu1>0</mu1>
-    <mu2>0</mu2>
-    <material>Gazebo/Black</material>
-  </gazebo>
-  <gazebo reference="fake_right_wheel">
-    <mu1>0</mu1>
-    <mu2>0</mu2>
-    <material>Gazebo/Black</material>
-  </gazebo>
 </robot>

File: simulation/ros2_ws_hex/src/hexapod_description/urdf/hexapod_leg.urdf.xacro (robot description, xacro)
@@ -14,4 +14,5 @@
        <visual>
          <origin xyz="-0.001140 0.000016 -0.002812" rpy="0 0 0"/>
+         <origin xyz="-0.001140 0.000016 1.002812" rpy="0 0 0"/>
          <geometry>
            <mesh filename="${meshes_file_direction}/platform.stl" scale="1.0 1.0 1.0"/>

File: simulation/ros2_ws_hex/src/hexapod_description/urdf/lidar.xacro (robot description, xacro)
@@ -1,3 +1,5 @@
 <?xml version="1.0"?>
+<!-- we wouldnt have a lidar in out hexapod it is just pretty similar to camera, that's why it was added like an example for futher development -->
+<!-- source - https://articulatedrobotics.xyz/tutorials/mobile-robot/hardware/lidar -->
 <robot xmlns:xacro="http://ros.org/wiki/xacro">
     <xacro:property name="prefix" value=""/>

Commit message: Loading the same model for Gazebo and MoveIt

File: simulation/ros2_ws_hex/src/hexapod_description/urdf/hexapod.urdf.xacro (robot description, xacro)
@@ -1,6 +1,8 @@
 <?xml version="1.0"?>
 <robot name="hexapod" xmlns:xacro="http://ros.org/wiki/xacro">
-    <xacro:arg name="use_gazebo" default="false" />
+    <!-- Declare the argument with a default value -->
+    <xacro:arg name="use_gazebo" default="true"/>
     <xacro:include filename="$(find hexapod_description)/urdf/hexapod_ee.urdf.xacro" />
+    <!-- Pass the argument value to the macro -->
     <xacro:hexapod_ee use_sim="true" prefix="" use_gazebo="$(arg use_gazebo)"/>
 </robot>

File: simulation/ros2_ws_hex/src/hexapod_description/urdf/hexapod_ee.urdf.xacro (robot description, xacro)
@@ -1,17 +1,23 @@
 <?xml version="1.0"?>
 <robot name="hexapod" xmlns:xacro="http://ros.org/wiki/xacro">
-  <xacro:arg name="use_sim" default="true" />
-  <xacro:arg name="prefix" default="" />
-  <xacro:include filename="$(find hexapod_description)/gazebo/hexapod.gazebo.xacro" />
-  <xacro:include filename="$(find hexapod_description)/urdf/hexapod_leg_ee.urdf.xacro" />
-  <xacro:include filename="$(find hexapod_description)/urdf/hexapod_gazebo.urdf.xacro" />
-  <xacro:include filename="$(find hexapod_description)/ros2_control/hexapod_system.ros2_control.xacro" />
-  <xacro:hexapod prefix="$(arg prefix)" />
-  <xacro:hexapod_gazebo prefix="$(arg prefix)" />
-  <xacro:hexapod_system use_sim="$(arg use_sim)" prefix="$(arg prefix)"/>
-  <gazebo>
-    <plugin filename="gz_ros2_control-system" name="gz_ros2_control::GazeboSimROS2ControlPlugin">
-      <parameters>$(find hex_gz)/config/gazebo_controller_manager.yaml</parameters>
-    </plugin>
-  </gazebo>
+  <xacro:macro name="hexapod_ee" params="use_sim prefix use_gazebo">
+    <xacro:arg name="use_sim" default="true" />
+    <xacro:arg name="prefix" default="" />
+    <xacro:include filename="$(find hexapod_description)/gazebo/hexapod.gazebo.xacro" />
+    <xacro:include filename="$(find hexapod_description)/urdf/hexapod_leg_ee.urdf.xacro" />
+    <xacro:include filename="$(find hexapod_description)/urdf/hexapod_gazebo.urdf.xacro" />
+    <!-- include pozycji początkowych -->
+    <!-- <xacro:include filename="$(find hexapod_description)/ros2_control/hexapod.ros2_control.xacro" /> -->
+    <xacro:include filename="$(find hexapod_moveit_config)/config/hexapod.ros2_control.xacro" />
+    <xacro:hexapod prefix="$(arg prefix)" />
+    <xacro:hexapod_gazebo prefix="$(arg prefix)" />
+    <gazebo>
+      <plugin filename="gz_ros2_control-system" name="gz_ros2_control::GazeboSimROS2ControlPlugin">
+        <parameters>$(find hex_gz)/config/gazebo_controller_manager.yaml</parameters>
+      </plugin>
+    </gazebo>
+    <!-- <xacro:hexapod_ros2_control name="FakeSystem" initial_positions_file="$(arg initial_positions_file)"/> -->
+    <!-- <xacro:hexapod_ros2_control use_sim="$(arg use_sim)" prefix="$(arg prefix)" initial_positions_file="$(find hexapod_description)/config/initial_positions.yaml"/>  -->
+    <xacro:hexapod_ros2_control name="hexapod" initial_positions_file="$(find hexapod_description)/config/initial_positions.yaml" use_gazebo="${use_gazebo}"/>
+  </xacro:macro>
 </robot>

File: simulation/ros2_ws_hex/src/hexapod_moveit_config/config/hexapod.ros2_control.xacro (robot description, xacro)
@@ -1,11 +1,21 @@
 <?xml version="1.0"?>
 <robot xmlns:xacro="http://www.ros.org/wiki/xacro">
-    <xacro:macro name="hexapod_ros2_control" params="name initial_positions_file">
+    <xacro:macro name="hexapod_ros2_control" params="name initial_positions_file use_gazebo">
         <xacro:property name="initial_positions" value="${xacro.load_yaml(initial_positions_file)['initial_positions']}"/>
         <ros2_control name="${name}" type="system">
+        <xacro:if value="${use_gazebo}">
             <hardware>
                 <!-- By default, set up controllers for simulation. This won't work on real hardware -->
+                <plugin>gz_ros2_control/GazeboSimSystem</plugin>
+                <!-- <plugin>mock_components/GenericSystem</plugin> -->
+            </hardware>
+        </xacro:if>
+        <xacro:unless value="${use_gazebo}">
+            <hardware>
+                <!-- By default, set up controllers for simulation. This won't work on real hardware -->
+                <!-- <plugin>gz_ros2_control/GazeboSimSystem</plugin> -->
                 <plugin>mock_components/GenericSystem</plugin>
             </hardware>
+        </xacro:unless>
             <!-- Leg 1 joints -->
             <joint name="joint1_1">
