Commit message: Update hexapod_leg_ee.urdf.xacro
Adding code that may be helpful in starting leg position

File: simulation/ros2_ws_hex/src/hexapod_description/urdf/hexapod_leg_ee.urdf.xacro (robot description, xacro)
@@ -119,5 +119,5 @@
       <parent link="${prefix}link3_1"/>
       <child link="${prefix}link4_1"/>
-      <origin xyz="-0.054636	0.071451	0.00505" rpy="0 0 0"/>
+      <origin xyz="-0.054636	0.071451	0.00505" rpy="1.4072 0 0"/>
       <axis xyz="-0.6074290528 -0.794374 0"/>
       <limit effort="5.0" velocity="1.0" lower="0" upper="1.570796327"/>
@@ -232,5 +232,5 @@
       <parent link="${prefix}link3_2"/>
       <child link="${prefix}link4_2"/>
-      <origin xyz="0.0	0.089946	0.00505" rpy="0 0 0"/>
+      <origin xyz="0.0	0.089946	0.00505" rpy="1.4072 0 0"/>
       <axis xyz="-1 0 0"/>
       <limit effort="5.0" velocity="1.0" lower="0" upper="1.570796327"/>
@@ -345,5 +345,5 @@
       <parent link="${prefix}link3_3"/>
       <child link="${prefix}link4_3"/>
-      <origin xyz="0.054636	0.071451	0.00505" rpy="0 0 0"/>
+      <origin xyz="0.054636	0.071451	0.00505" rpy="1.4072 0 0"/>
       <axis xyz="-0.794374 0.6074290528 0"/>
       <limit effort="5.0" velocity="1.0" lower="0" upper="1.570796327"/>
@@ -458,5 +458,5 @@
       <parent link="${prefix}link3_4"/>
       <child link="${prefix}link4_4"/>
-      <origin xyz="0.054636	-0.071451	0.00505" rpy="0 0 0"/>
+      <origin xyz="0.054636	-0.071451	0.00505" rpy="1.4072 0 0"/>
       <axis xyz="0.6074290528 0.794374 0"/>
       <limit effort="5.0" velocity="1.0" lower="0" upper="1.570796327"/>
@@ -571,5 +571,5 @@
       <parent link="${prefix}link3_5"/>
       <child link="${prefix}link4_5"/>
-      <origin xyz="0.0	-0.089946	0.00505" rpy="0 0 0"/>
+      <origin xyz="0.0	-0.089946	0.00505" rpy="1.4072 0 0"/>
       <axis xyz="1 0 0"/>
       <limit effort="5.0" velocity="1.0" lower="0" upper="1.570796327"/>
@@ -684,5 +684,5 @@
       <parent link="${prefix}link3_6"/>
       <child link="${prefix}link4_6"/>
-      <origin xyz="-0.054636	-0.071451	0.00505" rpy="0 0 0"/>
+      <origin xyz="-0.054636	-0.071451	0.00505" rpy="1.4072 0 0"/>
       <axis xyz="0.794374 -0.6074290528 0"/>
       <limit effort="5.0" velocity="1.0" lower="0" upper="1.570796327"/>
@@ -716,4 +716,5 @@
     </link>
     <!-- END EFFECTOR JOINT AND LINK -->
+<!--may be useful to set leg in starting position
     <joint name="${prefix}joint4_6" type="fixed">
       <parent link="${prefix}link4_6"/>
@@ -721,4 +722,40 @@
       <origin xyz="-0.099223	-0.130739	-0.000046" rpy="0 0 0"/>
     </joint>
+    <transmission name="${prefix}trans_joint1_6">
+      <type>transmission_interface/SimpleTransmission</type>
+      <joint name="${prefix}joint1_6">
+        <hardwareInterface>hardware_interface/PositionJointInterface</hardwareInterface>
+      </joint>
+      <actuator name="${prefix}motor1_6">
+        <hardwareInterface>hardware_interface/PositionJointInterface</hardwareInterface>
+        <mechanicalReduction>1.0</mechanicalReduction>
+      </actuator>
+    </transmission>
+    <transmission name="${prefix}trans_joint2_6">
+      <type>transmission_interface/SimpleTransmission</type>
+      <joint name="${prefix}joint2_6">
+        <hardwareInterface>hardware_interface/PositionJointInterface</hardwareInterface>
+      </joint>
+      <actuator name="${prefix}motor2_6">
+        <hardwareInterface>hardware_interface/PositionJointInterface</hardwareInterface>
+        <mechanicalReduction>1.0</mechanicalReduction>
+      </actuator>
+    </transmission>
+    <transmission name="${prefix}trans_joint3_6">
+      <type>transmission_interface/SimpleTransmission</type>
+      <joint name="${prefix}joint3_6">
+        <hardwareInterface>hardware_interface/PositionJointInterface</hardwareInterface>
+      </joint>
+      <actuator name="${prefix}motor3_6">
+        <hardwareInterface>hardware_interface/PositionJointInterface</hardwareInterface>
+        <mechanicalReduction>1.0</mechanicalReduction>
+      </actuator>
+    </transmission>
+    -->
+    <joint name="${prefix}joint4_6" type="fixed">
+      <parent link="${prefix}link4_6"/>
+      <child link="${prefix}link5_6"/>
+      <origin xyz="-0.099223	-0.130739	-0.000046" rpy="0 0 0"/>
+    </joint>
     <link name="${prefix}link5_6"/>
   </xacro:macro>

Commit message: fixing

File: simulation/ros2_ws_hex/src/hexapod_description/urdf/hexapod_leg_ee.urdf.xacro (robot description, xacro)
@@ -717,9 +717,4 @@
     <!-- END EFFECTOR JOINT AND LINK -->
 <!--may be useful to set leg in starting position
-    <joint name="${prefix}joint4_6" type="fixed">
-      <parent link="${prefix}link4_6"/>
-      <child link="${prefix}link5_6"/>
-      <origin xyz="-0.099223	-0.130739	-0.000046" rpy="0 0 0"/>
-    </joint>
     <transmission name="${prefix}trans_joint1_6">
       <type>transmission_interface/SimpleTransmission</type>

Commit message: dodanie pozycji + ruch w motion planning poprzez plik pythonowy

File: simulation/ros2_ws_hex/src/hexapod_description/urdf/hexapod_leg_ee.urdf.xacro (robot description, xacro)
@@ -85,5 +85,5 @@
       <child link="${prefix}link3_1"/>
       <origin xyz="-0.018864	0.024671	-0.020002" rpy="0 0 0"/>
-      <axis xyz="-0.6074290528 -0.794374 0"/>
+      <axis xyz="-0.7968540982 -0.6041717854 0"/>
       <limit effort="5.0" velocity="1.0" lower="-0.261799388" upper="1.308996939"/>
       <dynamics damping="0.1"/>
@@ -120,5 +120,5 @@
       <child link="${prefix}link4_1"/>
       <origin xyz="-0.054636	0.071451	0.00505" rpy="0 0 0"/>
-      <axis xyz="-0.6074290528 -0.794374 0"/>
+      <axis xyz="-0.7968540982 -0.6041717854 0"/>
       <limit effort="5.0" velocity="1.0" lower="0" upper="1.570796327"/>
       <dynamics damping="0.1"/>
@@ -459,5 +459,5 @@
       <child link="${prefix}link4_4"/>
       <origin xyz="0.054636	-0.071451	0.00505" rpy="0 0 0"/>
-      <axis xyz="0.6074290528 0.794374 0"/>
+      <axis xyz="0.794374 0.6074290528 0"/>
       <limit effort="5.0" velocity="1.0" lower="0" upper="1.570796327"/>
       <dynamics damping="0.1"/>

Commit message: split monolithic macro into modular macros

File: simulation/ros2_ws_hex/src/hexapod_description/urdf/hexapod_leg_ee.urdf.xacro (robot description, xacro)
@@ -6,107 +6,28 @@
    <xacro:property name="iyy" value="1.0"/>
    <xacro:property name="izz" value="1.0"/>
-   <xacro:macro name="hexapod" params="prefix=''">
-     <xacro:property
+   <xacro:property
        name="meshes_file_direction"
        value="package://hexapod_description/meshes"/>
-<!-- WORLD DEFINITION -->
-      <!-- <link name="world"/> -->
-      <!--
-      <joint name="${prefix}world_fixed" type="fixed">
+   <!-- Macro platformy -->
+   <xacro:macro name="platform_base" params="prefix">
+    <link name="${prefix}base_link">
+      <visual>
         <origin xyz="0 0 0" rpy="0 0 0"/>
-        <parent link="world"/>
-        <child link="${prefix}base_link"/>
-      </joint> -->
-<!-- PLATFORMA -->
-     <link name="${prefix}base_link">
-       <visual>
-         <origin xyz="0.0 0.0 0.0" rpy="0 0 0"/>
-         <geometry>
-           <mesh filename="${meshes_file_direction}/platform.stl" scale="1.0 1.0 1.0"/>
-         </geometry>
-         <material name="grey">
-           <color rgba="0.2 0.2 0.2 1"/>
-         </material>
-       </visual>
-       <collision>
-         <origin xyz="0.0 0.0 0.0" rpy="0 0 0"/>
-         <geometry>
-           <mesh filename="${meshes_file_direction}/hitbox_platform.stl" scale="1.0 1.0 1.0"/>
-         </geometry>
-       </collision>
-        <inertial>
-         <origin xyz="0.0 0.0 0.0" rpy="0.0 0.0 0.0"/>
-         <mass value="${base_mass}"/>
-         <inertia
-           ixx="${ixx}" ixy="0.0" ixz="0.0"
-           iyy="${iyy}" iyz="0.0"
-           izz="${izz}"/>
-       </inertial>
-     </link>
-  <!-- LEG 1!!!!!!!!!!!!!!!!!!!!!!!!!!!!!!!!!!!!!!!!!!!!!!!!!!!!!!!!!!!!!!! -->
-     <!-- PLATFORMA - UP_SECTION -->
-     <joint name="${prefix}joint1_1" type="revolute">
-       <parent link="${prefix}base_link"/>
-       <child link="${prefix}link2_1"/>
-       <origin xyz="-0.063746	0.067285	0.003274" rpy="0 0 0"/>
-       <axis xyz="0.0 0.0 1.0"/>
-       <limit effort="5.0" velocity="1.0" lower="-0.5236" upper="0.5236"/>
-       <dynamics damping="0.1"/>
-     </joint>
-   <!-- UP_SECTION -->
-     <link name="${prefix}link2_1">
-       <visual>
-         <origin xyz="-0.013611	0.016988 -0.000419" rpy="0 0 0"/>
-         <geometry>
-           <mesh filename="${meshes_file_direction}/1_leg_up.stl" scale="1.0 1.0 1.0"/>
-         </geometry>
-         <material name="grey">
-           <color rgba="0.2 0.2 0.2 1"/>
-         </material>
-       </visual>
-       <collision>
-         <origin xyz="-0.013611	0.016988 -0.000419" rpy="0 0 0"/>
-         <geometry>
-           <mesh filename="${meshes_file_direction}/hitbox_1_leg_up.stl" scale="1.0 1.0 1.0"/>
-         </geometry>
-       </collision>
-        <inertial>
-         <origin xyz="0.0 0.0 0.0" rpy="0.0 0.0 0.0"/>
-         <mass value="${wheel_mass}"/>
-         <inertia
-           ixx="${ixx}" ixy="0.0" ixz="0.0"
-           iyy="${iyy}" iyz="0.0"
-           izz="${izz}"/>
-       </inertial>
-     </link>
-     <!-- UP_SECTION - MID_SECTION -->
-     <joint name="${prefix}joint2_1" type="revolute">
-      <parent link="${prefix}link2_1"/>
-      <child link="${prefix}link3_1"/>
-      <origin xyz="-0.018864	0.024671	-0.020002" rpy="0 0 0"/>
-      <axis xyz="-0.7968540982 -0.6041717854 0"/>
-      <limit effort="5.0" velocity="1.0" lower="-0.261799388" upper="1.308996939"/>
-      <dynamics damping="0.1"/>
-    </joint>
-  <!-- MID_SECTION -->
-    <link name="${prefix}link3_1">
-      <visual>
-        <origin xyz="-0.024936	0.032658	0.000547" rpy="0 0 0"/>
-        <geometry>
-          <mesh filename="${meshes_file_direction}/1_leg_mid.stl" scale="1.0 1.0 1.0"/>
-        </geometry>
-        <material name="grey">
+        <geometry>
+          <mesh filename="${meshes_file_direction}/platform.stl" scale="1 1 1"/>
+        </geometry>
+        <material name="gray">
           <color rgba="0.2 0.2 0.2 1"/>
         </material>
       </visual>
       <collision>
-        <origin xyz="-0.024936	0.032658	0.000547" rpy="0 0 0"/>
-        <geometry>
-          <mesh filename="${meshes_file_direction}/hitbox_1_leg_mid.stl" scale="1.0 1.0 1.0"/>
+        <origin xyz="0 0 0" rpy="0 0 0"/>
+        <geometry>
+          <mesh filename="${meshes_file_direction}/hitbox_platform.stl" scale="1 1 1"/>
         </geometry>
       </collision>
-       <inertial>
-        <origin xyz="0.0 0.0 0.0" rpy="0.0 0.0 0.0"/>
-        <mass value="${wheel_mass}"/>
+      <inertial>
+        <origin xyz="0 0 0" rpy="0 0 0"/>
+        <mass value="${base_mass}"/>
         <inertia
           ixx="${ixx}" ixy="0.0" ixz="0.0"
@@ -115,19 +36,23 @@
       </inertial>
     </link>
-  <!-- MID_SECTION - DOWN_SECTION -->
-    <joint name="${prefix}joint3_1" type="revolute">
-      <parent link="${prefix}link3_1"/>
-      <child link="${prefix}link4_1"/>
-      <origin xyz="-0.054636	0.071451	0.00505" rpy="0 0 0"/>
-      <axis xyz="-0.7968540982 -0.6041717854 0"/>
-      <limit effort="5.0" velocity="1.0" lower="0" upper="1.570796327"/>
+  </xacro:macro>
+  <!-- Macro: Joint -->
+  <xacro:macro name="leg_joint" params="prefix joint_name parent_link child_link xyz axis lower upper">
+    <joint name="${joint_name}" type="revolute">
+      <parent link="${parent_link}"/>
+      <child link="${child_link}"/>
+      <origin xyz="${xyz}" rpy="0 0 0"/>
+      <axis xyz="${axis}"/>
+      <limit effort="5.0" velocity="1.0" lower="${lower}" upper="${upper}"/>
       <dynamics damping="0.1"/>
     </joint>
-  <!-- DOWN_SECTION -->
-    <link name="${prefix}link4_1">
+  </xacro:macro>
+  <!-- Macro: UP_SECTION -->
+  <xacro:macro name="upper_leg" params="prefix index xyz rpy">
+    <link name="${prefix}link2_${index}">
       <visual>
-        <origin xyz="-0.039176	0.05167	0" rpy="0 0 0"/>
-        <geometry>
-          <mesh filename="${meshes_file_direction}/1_leg_down.stl" scale="1.0 1.0 1.0"/>
+        <origin xyz="${xyz}" rpy="${rpy}"/>
+        <geometry>
+          <mesh filename="${meshes_file_direction}/${index}_leg_up.stl" scale="1.0 1.0 1.0"/>
         </geometry>
         <material name="grey">
@@ -136,41 +61,23 @@
       </visual>
       <collision>
-        <origin xyz="-0.039176	0.05167	0" rpy="0 0 0"/>
-        <geometry>
-          <mesh filename="${meshes_file_direction}/hitbox_1_leg_down.stl" scale="1.0 1.0 1.0"/>
+        <origin xyz="${xyz}" rpy="${rpy}"/>
+        <geometry>
+          <mesh filename="${meshes_file_direction}/hitbox_${index}_leg_up.stl" scale="1.0 1.0 1.0"/>
         </geometry>
       </collision>
-        <inertial>
-        <origin xyz="0.0        0.0 0.0" rpy="0.0 0.0 0.0"/>
+      <inertial>
+        <origin xyz="0.0 0.0 0.0" rpy="0.0 0.0 0.0"/>
         <mass value="${wheel_mass}"/>
-        <inertia
-          ixx="${ixx}" ixy="0.0" ixz="0.0"
-          iyy="${iyy}" iyz="0.0"
-          izz="${izz}"/>
+        <inertia ixx="${ixx}" ixy="0.0" ixz="0.0" iyy="${iyy}" iyz="0.0" izz="${izz}"/>
       </inertial>
     </link>
-    <!-- END EFFECTOR JOINT AND LINK -->
-    <joint name="${prefix}joint4_1" type="fixed">
-      <parent link="${prefix}link4_1"/>
-      <child link="${prefix}link5_1"/>
-      <origin xyz="-0.099587	0.130461	-0.000046" rpy="0 0 0"/>
-    </joint>
-    <link name="${prefix}link5_1"/>
-    <!-- LEG 2!!!!!!!!!!!!!!!!!!!!!!!!!!!!!!!!!!!!!!!!!!!!!!!!!!!!!!!!!!!!!!!!!!!!!!!1 -->
-     <!-- PLATFORMA - UP_SECTION -->
-     <joint name="${prefix}joint1_2" type="revolute">
-      <parent link="${prefix}base_link"/>
-      <child link="${prefix}link2_2"/>
-      <origin xyz="-0.005442	0.097816	0.003274" rpy="0 0 0"/>
-      <axis xyz="0.0 0.0 1.0"/>
-      <limit effort="5.0" velocity="1.0" lower="-0.5236" upper="0.5236"/>
-      <dynamics damping="0.1"/>
-    </joint>
-  <!-- UP_SECTION -->
-    <link name="${prefix}link2_2">
+  </xacro:macro>
+  <!-- Macro: MID_SECTION -->
+  <xacro:macro name="mid_leg" params="prefix index xyz rpy">
+    <link name="${prefix}link3_${index}">
       <visual>
-        <origin xyz="-0.000493	0.021762	-0.000419" rpy="0 0 0"/>
-        <geometry>
-          <mesh filename="${meshes_file_direction}/2_leg_up.stl" scale="1.0 1.0 1.0"/>
+        <origin xyz="${xyz}" rpy="${rpy}"/>
+        <geometry>
+          <mesh filename="${meshes_file_direction}/${index}_leg_mid.stl" scale="1.0 1.0 1.0"/>
         </geometry>
         <material name="grey">
@@ -179,33 +86,23 @@
       </visual>
       <collision>
-        <origin xyz="-0.000493	0.021762	-0.000419" rpy="0 0 0"/>
-        <geometry>
-          <mesh filename="${meshes_file_direction}/hitbox_2_leg_up.stl" scale="1.0 1.0 1.0"/>
+        <origin xyz="${xyz}" rpy="${rpy}"/>
+        <geometry>
+          <mesh filename="${meshes_file_direction}/hitbox_${index}_leg_mid.stl" scale="1.0 1.0 1.0"/>
         </geometry>
       </collision>
-       <inertial>
+      <inertial>
         <origin xyz="0.0 0.0 0.0" rpy="0.0 0.0 0.0"/>
         <mass value="${wheel_mass}"/>
-        <inertia
-          ixx="${ixx}" ixy="0.0" ixz="0.0"
-          iyy="${iyy}" iyz="0.0"
-          izz="${izz}"/>
+        <inertia ixx="${ixx}" ixy="0.0" ixz="0.0" iyy="${iyy}" iyz="0.0" izz="${izz}"/>
       </inertial>
     </link>
-  <!-- UP_SECTION - MID_SECTION -->
-    <joint name="${prefix}joint2_2" type="revolute">
-      <parent link="${prefix}link2_2"/>
-      <child link="${prefix}link3_2"/>
-      <origin xyz="0.0	0.031057	-0.020002" rpy="0 0 0"/>
-      <axis xyz="-1 0 0"/>
-      <limit effort="5.0" velocity="1.0" lower="-0.261799388" upper="1.308996939"/>
-      <dynamics damping="0.1"/>
-    </joint>
-  <!-- MID_SECTION -->
-    <link name="${prefix}link3_2">
+  </xacro:macro>
+  <!-- Macro: DOWN_SECTION -->
+  <xacro:macro name="lower_leg" params="prefix index xyz rpy">
+    <link name="${prefix}link4_${index}">
       <visual>
-        <origin xyz="0.0	0.041	0.000546" rpy="0 0 0"/>
-        <geometry>
-          <mesh filename="${meshes_file_direction}/2_leg_mid.stl" scale="1.0 1.0 1.0"/>
+        <origin xyz="${xyz}" rpy="${rpy}"/>
+        <geometry>
+          <mesh filename="${meshes_file_direction}/${index}_leg_down.stl" scale="1.0 1.0 1.0"/>
         </geometry>
         <material name="grey">
@@ -214,512 +111,230 @@
       </visual>
       <collision>
-        <origin xyz="0.0	0.041	0.000546" rpy="0 0 0"/>
-        <geometry>
-          <mesh filename="${meshes_file_direction}/hitbox_2_leg_mid.stl" scale="1.0 1.0 1.0"/>
+        <origin xyz="${xyz}" rpy="${rpy}"/>
+        <geometry>
+          <mesh filename="${meshes_file_direction}/hitbox_${index}_leg_down.stl" scale="1.0 1.0 1.0"/>
         </geometry>
       </collision>
-       <inertial>
+      <inertial>
         <origin xyz="0.0 0.0 0.0" rpy="0.0 0.0 0.0"/>
         <mass value="${wheel_mass}"/>
-        <inertia
-          ixx="${ixx}" ixy="0.0" ixz="0.0"
-          iyy="${iyy}" iyz="0.0"
-          izz="${izz}"/>
+        <inertia ixx="${ixx}" ixy="0.0" ixz="0.0" iyy="${iyy}" iyz="0.0" izz="${izz}"/>
       </inertial>
     </link>
-  <!-- MID_SECTION - DOWN_SECTION -->
-    <joint name="${prefix}joint3_2" type="revolute">
-      <parent link="${prefix}link3_2"/>
-      <child link="${prefix}link4_2"/>
-      <origin xyz="0.0	0.089946	0.00505" rpy="0 0 0"/>
-      <axis xyz="-1 0 0"/>
-      <limit effort="5.0" velocity="1.0" lower="0" upper="1.570796327"/>
-      <dynamics damping="0.1"/>
-    </joint>
-  <!-- DOWN_SECTION -->
-    <link name="${prefix}link4_2">
-      <visual>
-        <origin xyz="0.000265	0.064842	0.0" rpy="0 0 0"/>
-        <geometry>
-          <mesh filename="${meshes_file_direction}/2_leg_down.stl" scale="1.0 1.0 1.0"/>
-        </geometry>
-        <material name="grey">
-          <color rgba="0.2 0.2 0.2 1"/>
-        </material>
-      </visual>
-      <collision>
-        <origin xyz="0.000265	0.064842	0.0" rpy="0 0 0"/>
-        <geometry>
-          <mesh filename="${meshes_file_direction}/hitbox_2_leg_down.stl" scale="1.0 1.0 1.0"/>
-        </geometry>
-      </collision>
-       <inertial>
-        <origin xyz="0.0        0.0 0.0" rpy="0.0 0.0 0.0"/>
-        <mass value="${wheel_mass}"/>
-        <inertia
-          ixx="${ixx}" ixy="0.0" ixz="0.0"
-          iyy="${iyy}" iyz="0.0"
-          izz="${izz}"/>
-      </inertial>
-    </link>
-   <!-- END EFFECTOR JOINT AND LINK -->
-   <joint name="${prefix}joint4_2" type="fixed">
-    <parent link="${prefix}link4_2"/>
-    <child link="${prefix}link5_2"/>
-    <origin xyz="0.000147	0.164223	-0.000046" rpy="0 0 0"/>
+  </xacro:macro>
+<!-- Macro: Effector Joint -->
+<xacro:macro name="end_effector_joint" params="prefix index xyz rpy">
+  <joint name="${prefix}joint4_${index}" type="fixed">
+    <parent link="${prefix}link4_${index}"/>
+    <child link="${prefix}link5_${index}"/>
+    <origin xyz="${xyz}" rpy="${rpy}"/>
   </joint>
-  <link name="${prefix}link5_2"/>
- <!-- LEG 3!!!!!!!!!!!!!!!!!!!!!!!!!!!!!!!!!!!!!!!!!!!!!!!!!!!!!!!!!!!!!!! -->
-    <!-- PLATFORMA - UP_SECTION -->
-    <joint name="${prefix}joint1_3" type="revolute">
-      <parent link="${prefix}base_link"/>
-      <child link="${prefix}link2_3"/>
-      <origin xyz="0.055103	0.073938	0.003274" rpy="0 0 0"/>
-      <axis xyz="0.0 0.0 1.0"/>
-      <limit effort="5.0" velocity="1.0" lower="-0.5236" upper="0.5236"/>
-      <dynamics damping="0.1"/>
-    </joint>
-  <!-- UP_SECTION -->
-    <link name="${prefix}link2_3">
-      <visual>
-        <origin xyz="0.012827	0.017587 -0.000419" rpy="0 0 0"/>
-        <geometry>
-          <mesh filename="${meshes_file_direction}/3_leg_up.stl" scale="1.0 1.0 1.0"/>
-        </geometry>
-        <material name="grey">
-          <color rgba="0.2 0.2 0.2 1"/>
-        </material>
-      </visual>
-      <collision>
-        <origin xyz="0.012827	0.017587 -0.000419" rpy="0 0 0"/>
-        <geometry>
-          <mesh filename="${meshes_file_direction}/hitbox_3_leg_up.stl" scale="1.0 1.0 1.0"/>
-        </geometry>
-      </collision>
-       <inertial>
-        <origin xyz="0.0 0.0 0.0" rpy="0.0 0.0 0.0"/>
-        <mass value="${wheel_mass}"/>
-        <inertia
-          ixx="${ixx}" ixy="0.0" ixz="0.0"
-          iyy="${iyy}" iyz="0.0"
-          izz="${izz}"/>
-      </inertial>
-    </link>
-  <!-- UP_SECTION - MID_SECTION -->
-    <joint name="${prefix}joint2_3" type="revolute">
-      <parent link="${prefix}link2_3"/>
-      <child link="${prefix}link3_3"/>
-      <origin xyz="0.018864	0.024671	-0.020002" rpy="0 0 0"/>
-      <axis xyz="-0.794374 0.6074290528 0"/>
-      <limit effort="5.0" velocity="1.0" lower="-0.261799388" upper="1.308996939"/>
-      <dynamics damping="0.1"/>
-    </joint>
-  <!-- MID_SECTION -->
-    <link name="${prefix}link3_3">
-      <visual>
-        <origin xyz="0.024936	0.032658	0.000547" rpy="0 0 0"/>
-        <geometry>
-          <mesh filename="${meshes_file_direction}/3_leg_mid.stl" scale="1.0 1.0 1.0"/>
-        </geometry>
-        <material name="grey">
-          <color rgba="0.2 0.2 0.2 1"/>
-        </material>
-      </visual>
-      <collision>
-        <origin xyz="0.024936	0.032658	0.000547" rpy="0 0 0"/>
-        <geometry>
-          <mesh filename="${meshes_file_direction}/hitbox_3_leg_mid.stl" scale="1.0 1.0 1.0"/>
-        </geometry>
-      </collision>
-       <inertial>
-        <origin xyz="0.0 0.0 0.0" rpy="0.0 0.0 0.0"/>
-        <mass value="${wheel_mass}"/>
-        <inertia
-          ixx="${ixx}" ixy="0.0" ixz="0.0"
-          iyy="${iyy}" iyz="0.0"
-          izz="${izz}"/>
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