Commit message: I added simpler collision models, that are accepted by gazebo simulator. Now we use only one model for each leg.

File: simulation/ros2_ws_hex/src/hexapod_description/urdf/hexapod_leg_ee.urdf.xacro (robot description, xacro)
@@ -9,32 +9,33 @@
        name="meshes_file_direction"
        value="package://hexapod_description/meshes"/>
+   <!-- Include macro modeli kolizyjnych z prostych kształtów geometrycznych -->
+   <xacro:include filename="$(find hexapod_description)/meshes/platform_hitbox.xacro"/>
+   <xacro:include filename="$(find hexapod_description)/meshes/up_section_hitbox.xacro"/>
+   <xacro:include filename="$(find hexapod_description)/meshes/mid_section_hitbox.xacro"/>
+   <xacro:include filename="$(find hexapod_description)/meshes/down_section_hitbox.xacro"/>
    <!-- Macro platformy -->
-   <xacro:macro name="platform_base" params="prefix">
-    <link name="${prefix}base_link">
-      <visual>
-        <origin xyz="0 0 0" rpy="0 0 0"/>
-        <geometry>
-          <mesh filename="${meshes_file_direction}/platform.stl" scale="1 1 1"/>
-        </geometry>
-        <material name="gray">
-          <color rgba="0.2 0.2 0.2 1"/>
-        </material>
-      </visual>
-      <collision>
-        <origin xyz="0 0 0" rpy="0 0 0"/>
-        <geometry>
-          <mesh filename="${meshes_file_direction}/hitbox_platform.stl" scale="1 1 1"/>
-        </geometry>
-      </collision>
-      <inertial>
-        <origin xyz="0 0 0" rpy="0 0 0"/>
-        <mass value="${base_mass}"/>
-        <inertia
-          ixx="${ixx}" ixy="0.0" ixz="0.0"
-          iyy="${iyy}" iyz="0.0"
-          izz="${izz}"/>
-      </inertial>
-    </link>
-  </xacro:macro>
+    <xacro:macro name="platform_base" params="prefix">
+      <link name="${prefix}base_link">
+        <visual>
+          <origin xyz="0 0 0" rpy="0 0 0"/>
+          <geometry>
+            <mesh filename="${meshes_file_direction}/platform.stl" scale="1 1 1"/>
+          </geometry>
+          <material name="gray">
+            <color rgba="0.2 0.2 0.2 1"/>
+          </material>
+        </visual>
+        <!-- MODEL KOLIZYJNY -->
+        <xacro:platform_collision prefix="${prefix}" />
+        <inertial>
+          <origin xyz="0 0 0" rpy="0 0 0"/>
+          <mass value="${base_mass}"/>
+          <inertia
+            ixx="${ixx}" ixy="0.0" ixz="0.0"
+            iyy="${iyy}" iyz="0.0"
+            izz="${izz}"/>
+        </inertial>
+      </link>
+    </xacro:macro>
   <!-- Macro: Joint -->
   <xacro:macro name="leg_joint" params="prefix joint_name parent_link child_link xyz axis lower upper">
@@ -54,5 +55,5 @@
         <origin xyz="${xyz}" rpy="${rpy}"/>
         <geometry>
-          <mesh filename="${meshes_file_direction}/${index}_leg_up.stl" scale="1.0 1.0 1.0"/>
+          <mesh filename="${meshes_file_direction}/leg_up.stl" scale="1.0 1.0 1.0"/>
         </geometry>
         <material name="grey">
@@ -60,10 +61,6 @@
         </material>
       </visual>
-      <collision>
-        <origin xyz="${xyz}" rpy="${rpy}"/>
-        <geometry>
-          <mesh filename="${meshes_file_direction}/hitbox_${index}_leg_up.stl" scale="1.0 1.0 1.0"/>
-        </geometry>
-      </collision>
+      <!-- MODEL KOLIZYJNY -->
+      <xacro:upper_leg_collision prefix="${prefix}" position="${xyz}" rotation="${rpy}"/>
       <inertial>
         <origin xyz="0.0 0.0 0.0" rpy="0.0 0.0 0.0"/>
@@ -79,5 +76,5 @@
         <origin xyz="${xyz}" rpy="${rpy}"/>
         <geometry>
-          <mesh filename="${meshes_file_direction}/${index}_leg_mid.stl" scale="1.0 1.0 1.0"/>
+          <mesh filename="${meshes_file_direction}/leg_mid.stl" scale="1.0 1.0 1.0"/>
         </geometry>
         <material name="grey">
@@ -85,10 +82,6 @@
         </material>
       </visual>
-      <collision>
-        <origin xyz="${xyz}" rpy="${rpy}"/>
-        <geometry>
-          <mesh filename="${meshes_file_direction}/hitbox_${index}_leg_mid.stl" scale="1.0 1.0 1.0"/>
-        </geometry>
-      </collision>
+      <!-- MODEL KOLIZYJNY -->
+      <xacro:mid_leg_collision prefix="${prefix}" position="${xyz}" rotation="${rpy}"/>
       <inertial>
         <origin xyz="0.0 0.0 0.0" rpy="0.0 0.0 0.0"/>
@@ -104,5 +97,5 @@
         <origin xyz="${xyz}" rpy="${rpy}"/>
         <geometry>
-          <mesh filename="${meshes_file_direction}/${index}_leg_down.stl" scale="1.0 1.0 1.0"/>
+          <mesh filename="${meshes_file_direction}/leg_down.stl" scale="1.0 1.0 1.0"/>
         </geometry>
         <material name="grey">
@@ -110,10 +103,6 @@
         </material>
       </visual>
-      <collision>
-        <origin xyz="${xyz}" rpy="${rpy}"/>
-        <geometry>
-          <mesh filename="${meshes_file_direction}/hitbox_${index}_leg_down.stl" scale="1.0 1.0 1.0"/>
-        </geometry>
-      </collision>
+      <!-- MODEL KOLIZYJNY -->
+      <xacro:lower_leg_collision prefix="${prefix}" position="${xyz}" rotation="${rpy}"/>
       <inertial>
         <origin xyz="0.0 0.0 0.0" rpy="0.0 0.0 0.0"/>
@@ -149,5 +138,5 @@
   lower="-0.5236"
   upper="0.5236" />
-<xacro:upper_leg prefix="${prefix}" index="1" xyz="-0.013611	0.016988 -0.000419" rpy="0 0 0" />
+  <xacro:upper_leg prefix="${prefix}" index="1" xyz="-0.013611	0.016988 -0.000419" rpy="0 0 0.654498469" />
 <xacro:leg_joint
   prefix="${prefix}"
@@ -159,5 +148,5 @@
   lower="-0.261799388"
   upper="1.308996939" />
-<xacro:mid_leg prefix="${prefix}" index="1" xyz="-0.024936	0.032658	0.000547" rpy="0 0 0" />
+<xacro:mid_leg prefix="${prefix}" index="1" xyz="-0.024936	0.032658	0.000547" rpy="0 0 0.654498469" />
 <xacro:leg_joint
   prefix="${prefix}"
@@ -169,5 +158,5 @@
   lower="0"
   upper="1.570796327" />
-<xacro:lower_leg prefix="${prefix}" index="1" xyz="-0.039176	0.05167	0" rpy="0 0 0" />
+<xacro:lower_leg prefix="${prefix}" index="1" xyz="-0.039176	0.05167	0" rpy="0 0 0.654498469" />
 <xacro:end_effector_joint prefix="${prefix}" index="1" xyz="-0.099587 0.130461 -0.000046" rpy="0 0 0"/>
 <xacro:end_effector_link prefix="${prefix}" index="1"/>
@@ -215,5 +204,5 @@
   lower="-0.5236"
   upper="0.5236"/>
-<xacro:upper_leg prefix="${prefix}" index="3" xyz="0.012827	0.017587 -0.000419" rpy="0 0 0"/>
+<xacro:upper_leg prefix="${prefix}" index="3" xyz="0.012827	0.017587 -0.000419" rpy="0 0 -0.654498469"/>
 <xacro:leg_joint
   prefix="${prefix}"
@@ -225,5 +214,5 @@
   lower="-0.261799388"
   upper="1.308996939"/>
-<xacro:mid_leg prefix="${prefix}" index="3" xyz="0.024936	0.032658	0.000547" rpy="0 0 0"/>
+<xacro:mid_leg prefix="${prefix}" index="3" xyz="0.024936	0.032658	0.000547" rpy="0 0 -0.654498469"/>
 <xacro:leg_joint
   prefix="${prefix}"
@@ -235,5 +224,5 @@
   lower="0"
   upper="1.570796327"/>
-<xacro:lower_leg prefix="${prefix}" index="3" xyz="0.039176	0.05167	0" rpy="0 0 0"/>
+<xacro:lower_leg prefix="${prefix}" index="3" xyz="0.039176	0.05167	0" rpy="0 0 -0.654498469"/>
 <xacro:end_effector_joint prefix="${prefix}" index="3" xyz="0.099252	0.130694	-0.000046" rpy="0 0 0"/>
 <xacro:end_effector_link prefix="${prefix}" index="3"/>
@@ -248,5 +237,5 @@
   lower="-0.5236"
   upper="0.5236"/>
-<xacro:upper_leg prefix="${prefix}" index="4" xyz="0.013611	-0.016988 -0.000419" rpy="0 0 0"/>
+<xacro:upper_leg prefix="${prefix}" index="4" xyz="0.013611	-0.016988 -0.000419" rpy="0 0 3.796091123"/>
 <xacro:leg_joint
   prefix="${prefix}"
@@ -258,5 +247,5 @@
   lower="-0.261799388"
   upper="1.308996939"/>
-<xacro:mid_leg prefix="${prefix}" index="4" xyz="0.024936	-0.032658	0.000547" rpy="0 0 0"/>
+<xacro:mid_leg prefix="${prefix}" index="4" xyz="0.024936	-0.032658	0.000547" rpy="0 0 3.796091123"/>
 <xacro:leg_joint
   prefix="${prefix}"
@@ -268,5 +257,5 @@
   lower="0"
   upper="1.570796327"/>
-<xacro:lower_leg prefix="${prefix}" index="4" xyz="0.039176	-0.05167	0" rpy="0 0 0"/>
+<xacro:lower_leg prefix="${prefix}" index="4" xyz="0.039176	-0.05167	0" rpy="0 0 3.796091123"/>
 <xacro:end_effector_joint prefix="${prefix}" index="4" xyz="0.099758	-0.130448	-0.000046" rpy="0 0 0"/>
 <xacro:end_effector_link prefix="${prefix}" index="4"/>
@@ -281,5 +270,5 @@
   lower="-0.5236"
   upper="0.5236"/>
-<xacro:upper_leg prefix="${prefix}" index="5" xyz="0.000493	-0.021762	-0.000419" rpy="0 0 0"/>
+<xacro:upper_leg prefix="${prefix}" index="5" xyz="0.000493	-0.021762	-0.000419" rpy="0 0 3.141592654"/>
 <xacro:leg_joint
   prefix="${prefix}"
@@ -291,5 +280,5 @@
   lower="-0.261799388"
   upper="1.308996939"/>
-<xacro:mid_leg prefix="${prefix}" index="5" xyz="0.0	-0.041	0.000546" rpy="0 0 0"/>
+<xacro:mid_leg prefix="${prefix}" index="5" xyz="0.0	-0.041	0.000546" rpy="0 0 3.141592654"/>
 <xacro:leg_joint
   prefix="${prefix}"
@@ -301,5 +290,5 @@
   lower="0"
   upper="1.570796327"/>
-<xacro:lower_leg prefix="${prefix}" index="5" xyz="-0.000265	-0.064842	0.0" rpy="0 0 0"/>
+<xacro:lower_leg prefix="${prefix}" index="5" xyz="-0.000265	-0.064842	0.0" rpy="0 0 3.141592654"/>
 <xacro:end_effector_joint prefix="${prefix}" index="5" xyz="-0.000051	-0.164207	-0.000046" rpy="0 0 0"/>
 <xacro:end_effector_link prefix="${prefix}" index="5"/>
@@ -314,5 +303,5 @@
   lower="-0.5236"
   upper="0.5236"/>
-<xacro:upper_leg prefix="${prefix}" index="6" xyz="-0.012827	-0.017588 -0.000419" rpy="0 0 0"/>
+<xacro:upper_leg prefix="${prefix}" index="6" xyz="-0.012827	-0.017588 -0.000419" rpy="0 0 2.487094184"/>
 <xacro:leg_joint
   prefix="${prefix}"
@@ -324,5 +313,5 @@
   lower="-0.261799388"
   upper="1.308996939"/>
-<xacro:mid_leg prefix="${prefix}" index="6" xyz="-0.024936	-0.032658	0.000547" rpy="0 0 0"/>
+<xacro:mid_leg prefix="${prefix}" index="6" xyz="-0.024936	-0.032658	0.000547" rpy="0 0 2.487094184"/>
 <xacro:leg_joint
   prefix="${prefix}"
@@ -334,5 +323,5 @@
   lower="0"
   upper="1.570796327"/>
-<xacro:lower_leg prefix="${prefix}" index="6" xyz="-0.039176	-0.05167	0" rpy="0 0 0"/>
+<xacro:lower_leg prefix="${prefix}" index="6" xyz="-0.039176	-0.05167	0" rpy="0 0 2.487094184"/>
 <xacro:end_effector_joint prefix="${prefix}" index="6" xyz="-0.099223	-0.130739	-0.000046" rpy="0 0 0"/>
 <xacro:end_effector_link prefix="${prefix}" index="6"/>

Commit message: Corrected few physics properties

File: simulation/ros2_ws_hex/src/hexapod_description/urdf/hexapod_leg_ee.urdf.xacro (robot description, xacro)
@@ -1,9 +1,11 @@
 <?xml version="1.0"?>
  <robot xmlns:xacro="http://www.ros.org/wiki/xacro">
-   <xacro:property name="base_mass" value="4.6" />
-   <xacro:property name="wheel_mass" value="1.0" />
-   <xacro:property name="ixx" value="1.0"/>
-   <xacro:property name="iyy" value="1.0"/>
-   <xacro:property name="izz" value="1.0"/>
+   <xacro:property name="platform_mass" value="0.3" />
+   <xacro:property name="up_section_mass" value="0.1" />
+   <xacro:property name="mid_section_mass" value="0.1" />
+   <xacro:property name="down_section_mass" value="0.1" />
+   <xacro:property name="ixx" value="0.001"/>
+   <xacro:property name="iyy" value="0.001"/>
+   <xacro:property name="izz" value="0.001"/>
    <xacro:property
        name="meshes_file_direction"
@@ -30,5 +32,5 @@
         <inertial>
           <origin xyz="0 0 0" rpy="0 0 0"/>
-          <mass value="${base_mass}"/>
+          <mass value="${platform_mass}"/>
           <inertia
             ixx="${ixx}" ixy="0.0" ixz="0.0"
@@ -64,6 +66,6 @@
       <xacro:upper_leg_collision prefix="${prefix}" position="${xyz}" rotation="${rpy}"/>
       <inertial>
-        <origin xyz="0.0 0.0 0.0" rpy="0.0 0.0 0.0"/>
-        <mass value="${wheel_mass}"/>
+        <origin xyz="${xyz}" rpy="0.0 0.0 0.0"/>
+        <mass value="${up_section_mass}"/>
         <inertia ixx="${ixx}" ixy="0.0" ixz="0.0" iyy="${iyy}" iyz="0.0" izz="${izz}"/>
       </inertial>
@@ -85,6 +87,6 @@
       <xacro:mid_leg_collision prefix="${prefix}" position="${xyz}" rotation="${rpy}"/>
       <inertial>
-        <origin xyz="0.0 0.0 0.0" rpy="0.0 0.0 0.0"/>
-        <mass value="${wheel_mass}"/>
+        <origin xyz="${xyz}" rpy="${rpy}"/>
+        <mass value="${mid_section_mass}"/>
         <inertia ixx="${ixx}" ixy="0.0" ixz="0.0" iyy="${iyy}" iyz="0.0" izz="${izz}"/>
       </inertial>
@@ -106,6 +108,6 @@
       <xacro:lower_leg_collision prefix="${prefix}" position="${xyz}" rotation="${rpy}"/>
       <inertial>
-        <origin xyz="0.0 0.0 0.0" rpy="0.0 0.0 0.0"/>
-        <mass value="${wheel_mass}"/>
+        <origin xxyz="${xyz}" rpy="${rpy}"/>
+        <mass value="${down_section_mass}"/>
         <inertia ixx="${ixx}" ixy="0.0" ixz="0.0" iyy="${iyy}" iyz="0.0" izz="${izz}"/>
       </inertial>
