Commit message: adjusting xacro to inertia, adding inertia to xacro

File: simulation/ros2_ws_hex/src/hexapod_description/urdf/hexapod_leg_ee.urdf.xacro (robot description, xacro)
@@ -5,7 +5,4 @@
    <xacro:property name="mid_section_mass" value="0.1" />
    <xacro:property name="down_section_mass" value="0.1" />
-   <xacro:property name="ixx" value="0.001"/>
-   <xacro:property name="iyy" value="0.001"/>
-   <xacro:property name="izz" value="0.001"/>
    <xacro:property
        name="meshes_file_direction"
@@ -17,5 +14,5 @@
    <xacro:include filename="$(find hexapod_description)/collision/down_section_hitbox.xacro"/>
    <!-- Macro platformy -->
-    <xacro:macro name="platform_base" params="prefix">
+    <xacro:macro name="platform_base" params="prefix ixx ixy ixz iyy iyz izz">
       <link name="${prefix}base_link">
         <visual>
@@ -34,6 +31,6 @@
           <mass value="${platform_mass}"/>
           <inertia
-            ixx="${ixx}" ixy="0.0" ixz="0.0"
-            iyy="${iyy}" iyz="0.0"
+            ixx="${ixx}" ixy="${ixy}" ixz="${ixz}"
+            iyy="${iyy}" iyz="${iyz}"
             izz="${izz}"/>
         </inertial>
@@ -52,5 +49,5 @@
   </xacro:macro>
   <!-- Macro: UP_SECTION -->
-  <xacro:macro name="upper_leg" params="prefix index xyz rpy">
+  <xacro:macro name="upper_leg" params="prefix index xyz rpy ixx ixy ixz iyy iyz izz">
     <link name="${prefix}link2_${index}">
       <visual>
@@ -68,10 +65,10 @@
         <origin xyz="${xyz}" rpy="0.0 0.0 0.0"/>
         <mass value="${up_section_mass}"/>
-        <inertia ixx="${ixx}" ixy="0.0" ixz="0.0" iyy="${iyy}" iyz="0.0" izz="${izz}"/>
+        <inertia ixx="${ixx}" ixy="${ixy}" ixz="${ixz}" iyy="${iyy}" iyz="${iyz}" izz="${izz}"/>
       </inertial>
     </link>
   </xacro:macro>
   <!-- Macro: MID_SECTION -->
-  <xacro:macro name="mid_leg" params="prefix index xyz rpy">
+  <xacro:macro name="mid_leg" params="prefix index xyz rpy ixx ixy ixz iyy iyz izz">
     <link name="${prefix}link3_${index}">
       <visual>
@@ -89,10 +86,10 @@
         <origin xyz="${xyz}" rpy="${rpy}"/>
         <mass value="${mid_section_mass}"/>
-        <inertia ixx="${ixx}" ixy="0.0" ixz="0.0" iyy="${iyy}" iyz="0.0" izz="${izz}"/>
+        <inertia ixx="${ixx}" ixy="${ixy}" ixz="${ixz}" iyy="${iyy}" iyz="${iyz}" izz="${izz}"/>
       </inertial>
     </link>
   </xacro:macro>
   <!-- Macro: DOWN_SECTION -->
-  <xacro:macro name="lower_leg" params="prefix index xyz rpy">
+  <xacro:macro name="lower_leg" params="prefix index xyz rpy ixx ixy ixz iyy iyz izz">
     <link name="${prefix}link4_${index}">
       <visual>
@@ -110,5 +107,5 @@
         <origin xxyz="${xyz}" rpy="${rpy}"/>
         <mass value="${down_section_mass}"/>
-        <inertia ixx="${ixx}" ixy="0.0" ixz="0.0" iyy="${iyy}" iyz="0.0" izz="${izz}"/>
+        <inertia ixx="${ixx}" ixy="${ixy}" ixz="${ixz}" iyy="${iyy}" iyz="${iyz}" izz="${izz}"/>
       </inertial>
     </link>
@@ -129,5 +126,12 @@
 <xacro:macro name="hexapod" params="prefix=''">
   <!-- Platform -->
-  <xacro:platform_base prefix="${prefix}" />
+<xacro:platform_base
+  prefix="${prefix}"
+  ixx="2.752506e-03"
+  ixy="2.768026e-08"
+  ixz="-1.305478e-06"
+  iyy="1.430780e-03"
+  iyz="1.593686e-10"
+  izz="3.895841e-03"/>
 <!-- LEG 1 -->
 <xacro:leg_joint
@@ -140,5 +144,15 @@
   lower="-0.5236"
   upper="0.5236" />
-  <xacro:upper_leg prefix="${prefix}" index="1" xyz="-0.013611	0.016988 -0.000419" rpy="0 0 0.654498469" />
+<xacro:upper_leg
+  prefix="${prefix}"
+  index="1"
+  xyz="-0.013611	0.016988 -0.000419"
+  rpy="0 0 0.654498469"
+  ixx="2.568568e-05"
+  ixy="7.190815e-06"
+  ixz="-4.383121e-07"
+  iyy="1.022635e-05"
+  iyz="-5.320311e-07"
+  izz="2.781267e-05"/>
 <xacro:leg_joint
   prefix="${prefix}"
@@ -150,5 +164,14 @@
   lower="-0.261799388"
   upper="1.308996939" />
-<xacro:mid_leg prefix="${prefix}" index="1" xyz="-0.024936	0.032658	0.000547" rpy="0 0 0.654498469" />
+<xacro:mid_leg
+  prefix="${prefix}"
+  index="1" xyz="-0.024936	0.032658	0.000547"
+  rpy="0 0 0.654498469"
+  ixx="1.071725e-04"
+  ixy="4.118637e-05"
+  ixz="6.741401e-07"
+  iyy="3.853424e-05"
+  iyz="-2.945627e-06"
+  izz="1.379702e-04"/>
 <xacro:leg_joint
   prefix="${prefix}"
@@ -160,5 +183,15 @@
   lower="0"
   upper="1.570796327" />
-<xacro:lower_leg prefix="${prefix}" index="1" xyz="-0.039176	0.05167	0" rpy="0 0 0.654498469" />
+<xacro:lower_leg
+  prefix="${prefix}"
+  index="1"
+  xyz="-0.039176	0.05167	0"
+  rpy="0 0 0.654498469"
+  ixx="2.892772e-04"
+  ixy="1.082271e-04"
+  ixz="4.221544e-08"
+  iyy="8.850525e-05"
+  iyz="-1.141746e-07"
+  izz="3.712638e-04"/>
 <xacro:end_effector_joint prefix="${prefix}" index="1" xyz="-0.099587 0.130461 -0.000046" rpy="0 0 0"/>
 <xacro:end_effector_link prefix="${prefix}" index="1"/>
@@ -173,5 +206,15 @@
   lower="-0.5236"
   upper="0.5236"/>
-<xacro:upper_leg prefix="${prefix}" index="2" xyz="-0.000493	0.021762	-0.000419" rpy="0 0 0"/>
+<xacro:upper_leg
+  prefix="${prefix}"
+  index="2"
+  xyz="-0.000493	0.021762	-0.000419"
+  rpy="0 0 0"
+  ixx="3.123539e-05"
+  ixy="5.760573e-07"
+  ixz="-2.734288e-07"
+  iyy="4.675870e-06"
+  iyz="-4.720256e-07"
+  izz="2.781190e-05"/>
 <xacro:leg_joint
   prefix="${prefix}"
@@ -183,5 +226,15 @@
   lower="-0.261799388"
   upper="1.308996939"/>
-<xacro:mid_leg prefix="${prefix}" index="2" xyz="0.0	0.041	0.000546" rpy="0 0 0"/>
+<xacro:mid_leg
+  prefix="${prefix}"
+  index="2"
+  xyz="0.0	0.041	0.000546"
+  rpy="0 0 0"
+  ixx="1.372807e-04"
+  ixy="1.282678e-06"
+  ixz="5.615442e-09"
+  iyy="8.065921e-06"
+  iyz="-3.167264e-06"
+  izz="1.376103e-04"/>
 <xacro:leg_joint
   prefix="${prefix}"
@@ -193,5 +246,15 @@
   lower="0"
   upper="1.570796327"/>
-<xacro:lower_leg prefix="${prefix}" index="2" xyz="0.000265	0.064842	0.0" rpy="0 0 0"/>
+<xacro:lower_leg
+  prefix="${prefix}"
+  index="2"
+  xyz="0.000265	0.064842	0.0"
+  rpy="0 0 0"
+  ixx="3.706160e-04"
+  ixy="3.252977e-08"
+  ixz="4.221449e-08"
+  iyy="7.167254e-06"
+  iyz="-1.141749e-07"
+  izz="3.712646e-04"/>
 <xacro:end_effector_joint prefix="${prefix}" index="2" xyz="0.000147	0.164223	-0.000046" rpy="0 0 0"/>
 <xacro:end_effector_link prefix="${prefix}" index="2"/>
@@ -206,5 +269,15 @@
   lower="-0.5236"
   upper="0.5236"/>
-<xacro:upper_leg prefix="${prefix}" index="3" xyz="0.012827	0.017587 -0.000419" rpy="0 0 -0.654498469"/>
+<xacro:upper_leg
+  prefix="${prefix}"
+  index="3"
+  xyz="0.012827	0.017587 -0.000419"
+  rpy="0 0 -0.654498469"
+  ixx="2.630698e-05"
+  ixy="-6.513359e-06"
+  ixz="-1.060066e-07"
+  iyy="9.604546e-06"
+  iyz="-5.245021e-07"
+  izz="2.781217e-05"/>
 <xacro:leg_joint
   prefix="${prefix}"
@@ -216,5 +289,15 @@
   lower="-0.261799388"
   upper="1.308996939"/>
-<xacro:mid_leg prefix="${prefix}" index="3" xyz="0.024936	0.032658	0.000547" rpy="0 0 -0.654498469"/>
+<xacro:mid_leg
+  prefix="${prefix}"
+  index="3"
+  xyz="0.024936	0.032658	0.000547"
+  rpy="0 0 -0.654498469"
+  ixx="1.071725e-04"
+  ixy="-3.862097e-05"
+  ixz="-6.629092e-07"
+  iyy="3.853451e-05"
+  iyz="-2.945627e-06"
+  izz="1.379705e-04"/>
 <xacro:leg_joint
   prefix="${prefix}"
@@ -226,5 +309,15 @@
   lower="0"
   upper="1.570796327"/>
-<xacro:lower_leg prefix="${prefix}" index="3" xyz="0.039176	0.05167	0" rpy="0 0 -0.654498469"/>
+<xacro:lower_leg
+  prefix="${prefix}"
+  index="3"
+  xyz="0.039176	0.05167	0"
+  rpy="0 0 -0.654498469"
+  ixx="2.892772e-04"
+  ixy="-1.063404e-04"
+  ixz="4.221354e-08"
+  iyy="8.850626e-05"
+  iyz="-1.141746e-07"
+  izz="3.712648e-04"/>
 <xacro:end_effector_joint prefix="${prefix}" index="3" xyz="0.099252	0.130694	-0.000046" rpy="0 0 0"/>
 <xacro:end_effector_link prefix="${prefix}" index="3"/>
@@ -239,5 +332,15 @@
   lower="-0.5236"
   upper="0.5236"/>
-<xacro:upper_leg prefix="${prefix}" index="4" xyz="0.013611	-0.016988 -0.000419" rpy="0 0 3.796091123"/>
+<xacro:upper_leg
+  prefix="${prefix}"
+  index="4"
+  xyz="0.013611	-0.016988 -0.000419"
+  rpy="0 0 3.796091123"
+  ixx="2.568617e-05"
+  ixy="7.191023e-06"
+  ixz="-9.615233e-08"
+  iyy="1.022637e-05"
+  iyz="-9.590835e-07"
+  izz="2.781317e-05"/>
 <xacro:leg_joint
   prefix="${prefix}"
@@ -249,5 +352,15 @@
   lower="-0.261799388"
   upper="1.308996939"/>
-<xacro:mid_leg prefix="${prefix}" index="4" xyz="0.024936	-0.032658	0.000547" rpy="0 0 3.796091123"/>
+<xacro:mid_leg
+  prefix="${prefix}"
+  index="4"
+  xyz="0.024936	-0.032658	0.000547"
+  rpy="0 0 3.796091123"
+  ixx="1.071723e-04"
+  ixy="4.118647e-05"
+  ixz="-6.629092e-07"
+  iyy="3.853451e-05"
+  iyz="-1.194530e-06"
+  izz="1.379703e-04"/>
 <xacro:leg_joint
   prefix="${prefix}"
@@ -259,5 +372,15 @@
   lower="0"
   upper="1.570796327"/>
-<xacro:lower_leg prefix="${prefix}" index="4" xyz="0.039176	-0.05167	0" rpy="0 0 3.796091123"/>
+<xacro:lower_leg
+  prefix="${prefix}"
+  index="4"
+  xyz="0.039176	-0.05167	0"
+  rpy="0 0 3.796091123"
+  ixx="2.892779e-04"
+  ixy="1.082280e-04"
+  ixz="4.221354e-08"
+  iyy="8.850626e-05"
+  iyz="-1.141720e-07"
+  izz="3.712655e-04"/>
 <xacro:end_effector_joint prefix="${prefix}" index="4" xyz="0.099758	-0.130448	-0.000046" rpy="0 0 0"/>
 <xacro:end_effector_link prefix="${prefix}" index="4"/>
@@ -272,5 +395,15 @@
   lower="-0.5236"
   upper="0.5236"/>
-<xacro:upper_leg prefix="${prefix}" index="5" xyz="0.000493	-0.021762	-0.000419" rpy="0 0 3.141592654"/>
+<xacro:upper_leg
+  prefix="${prefix}"
+  index="5"
+  xyz="0.000493	-0.021762	-0.000419"
+  rpy="0 0 3.141592654"
+  ixx="3.123601e-05"
+  ixy="5.760804e-07"
+  ixz="-2.610356e-07"
+  iyy="4.675871e-06"
+  iyz="-1.019089e-06"
+  izz="2.781252e-05"/>
 <xacro:leg_joint
   prefix="${prefix}"
@@ -282,5 +415,15 @@
   lower="-0.261799388"
   upper="1.308996939"/>
-<xacro:mid_leg prefix="${prefix}" index="5" xyz="0.0	-0.041	0.000546" rpy="0 0 3.141592654"/>
+<xacro:mid_leg
+  prefix="${prefix}"
+  index="5"
+  xyz="0.0	-0.041	0.000546"
+  rpy="0 0 3.141592654"
+  ixx="1.372805e-04"
+  ixy="1.282896e-06"
+  ixz="5.615442e-09"
+  iyy="8.065921e-06"
+  iyz="-9.728935e-07"
+  izz="1.376100e-04"/>
 <xacro:leg_joint
   prefix="${prefix}"
@@ -292,5 +435,15 @@
   lower="0"
   upper="1.570796327"/>
-<xacro:lower_leg prefix="${prefix}" index="5" xyz="-0.000265	-0.064842	0.0" rpy="0 0 3.141592654"/>
+<xacro:lower_leg
+  prefix="${prefix}"
+  index="5"
+  xyz="-0.000265	-0.064842	0.0"
+  rpy="0 0 3.141592654"
+  ixx="3.706168e-04"
+  ixy="3.335744e-08"
+  ixz="4.221450e-08"
+  iyy="7.167247e-06"
+  iyz="-1.141717e-07"
+  izz="3.712654e-04"/>
 <xacro:end_effector_joint prefix="${prefix}" index="5" xyz="-0.000051	-0.164207	-0.000046" rpy="0 0 0"/>
 <xacro:end_effector_link prefix="${prefix}" index="5"/>
@@ -305,5 +458,15 @@
   lower="-0.5236"
   upper="0.5236"/>
-<xacro:upper_leg prefix="${prefix}" index="6" xyz="-0.012827	-0.017588 -0.000419" rpy="0 0 2.487094184"/>
+<xacro:upper_leg
+  prefix="${prefix}"
+  index="6"
+  xyz="-0.012827	-0.017588 -0.000419"
+  rpy="0 0 2.487094184"
+  ixx="2.630854e-05"
+  ixy="-6.513915e-06"
+  ixz="-4.284578e-07"
+  iyy="9.604527e-06"
+  iyz="-9.666250e-07"
+  izz="2.781371e-05"/>
 <xacro:leg_joint
   prefix="${prefix}"
@@ -315,5 +478,15 @@
   lower="-0.261799388"
   upper="1.308996939"/>
-<xacro:mid_leg prefix="${prefix}" index="6" xyz="-0.024936	-0.032658	0.000547" rpy="0 0 2.487094184"/>
+<xacro:mid_leg
+  prefix="${prefix}"
+  index="6"
+  xyz="-0.024936	-0.032658	0.000547"
+  rpy="0 0 2.487094184"
+  ixx="1.071723e-04"
+  ixy="-3.862072e-05"
+  ixz="6.741401e-07"
+  iyy="3.853424e-05"
+  iyz="-1.194530e-06"
+  izz="1.379700e-04"/>
 <xacro:leg_joint
   prefix="${prefix}"
@@ -325,5 +498,15 @@
   lower="0"
   upper="1.570796327"/>
-<xacro:lower_leg prefix="${prefix}" index="6" xyz="-0.039176	-0.05167	0" rpy="0 0 2.487094184"/>
+<xacro:lower_leg
+  prefix="${prefix}"
+  index="6"
+  xyz="-0.039176	-0.05167	0"
+  rpy="0 0 2.487094184"
+  ixx="2.892779e-04"
+  ixy="-1.063400e-04"
+  ixz="4.221544e-08"
+  iyy="8.850525e-05"
+  iyz="-1.141720e-07"
+  izz="3.712645e-04"/>
 <xacro:end_effector_joint prefix="${prefix}" index="6" xyz="-0.099223	-0.130739	-0.000046" rpy="0 0 0"/>
 <xacro:end_effector_link prefix="${prefix}" index="6"/>
