Commit message: poprawiony motion planning w moveit, poprawiony gazebo.launch.py

File: simulation/ros2_ws_hex/src/hexapod_description/gazebo/hexapod.gazebo.xacro (robot description, xacro)
@@ -24,12 +24,60 @@
     </gazebo>
   </xacro:macro>
-  <xacro:Link reference="${prefix}link1"/>
-  <xacro:Link reference="${prefix}link2"/>
-  <xacro:Link reference="${prefix}link3"/>
-  <xacro:Link reference="${prefix}link4"/>
-  <!-- NALEŻY DOPISAĆ POZOSTAŁE LINKI ROBOTA, WAŻNE DO ALGORYTMÓW CHODZENIA -->
-  <xacro:SimpleTransmission trans="${prefix}trans1" joint="${prefix}joint1_1" actuator="${prefix}actuator1" />
-  <xacro:SimpleTransmission trans="${prefix}trans2" joint="${prefix}joint2_1" actuator="${prefix}actuator2" />
-  <xacro:SimpleTransmission trans="${prefix}trans3" joint="${prefix}joint3_1" actuator="${prefix}actuator3" />
+  <!-- Define links for all parts of the hexapod -->
+  <xacro:Link reference="${prefix}base_link"/>
+  <!-- Leg 1 links -->
+  <xacro:Link reference="${prefix}link1_1"/>
+  <xacro:Link reference="${prefix}link2_1"/>
+  <xacro:Link reference="${prefix}link3_1"/>
+  <xacro:Link reference="${prefix}link4_1"/>
+  <!-- Leg 2 links -->
+  <xacro:Link reference="${prefix}link1_2"/>
+  <xacro:Link reference="${prefix}link2_2"/>
+  <xacro:Link reference="${prefix}link3_2"/>
+  <xacro:Link reference="${prefix}link4_2"/>
+  <!-- Leg 3 links -->
+  <xacro:Link reference="${prefix}link1_3"/>
+  <xacro:Link reference="${prefix}link2_3"/>
+  <xacro:Link reference="${prefix}link3_3"/>
+  <xacro:Link reference="${prefix}link4_3"/>
+  <!-- Leg 4 links -->
+  <xacro:Link reference="${prefix}link1_4"/>
+  <xacro:Link reference="${prefix}link2_4"/>
+  <xacro:Link reference="${prefix}link3_4"/>
+  <xacro:Link reference="${prefix}link4_4"/>
+  <!-- Leg 5 links -->
+  <xacro:Link reference="${prefix}link1_5"/>
+  <xacro:Link reference="${prefix}link2_5"/>
+  <xacro:Link reference="${prefix}link3_5"/>
+  <xacro:Link reference="${prefix}link4_5"/>
+  <!-- Leg 6 links -->
+  <xacro:Link reference="${prefix}link1_6"/>
+  <xacro:Link reference="${prefix}link2_6"/>
+  <xacro:Link reference="${prefix}link3_6"/>
+  <xacro:Link reference="${prefix}link4_6"/>
+  <!-- Leg 1 Transmissions -->
+  <xacro:SimpleTransmission trans="${prefix}leg1_trans1" joint="${prefix}joint1_1" actuator="${prefix}leg1_motor1" />
+  <xacro:SimpleTransmission trans="${prefix}leg1_trans2" joint="${prefix}joint2_1" actuator="${prefix}leg1_motor2" />
+  <xacro:SimpleTransmission trans="${prefix}leg1_trans3" joint="${prefix}joint3_1" actuator="${prefix}leg1_motor3" />
+  <!-- Leg 2 Transmissions -->
+  <xacro:SimpleTransmission trans="${prefix}leg2_trans1" joint="${prefix}joint1_2" actuator="${prefix}leg2_motor1" />
+  <xacro:SimpleTransmission trans="${prefix}leg2_trans2" joint="${prefix}joint2_2" actuator="${prefix}leg2_motor2" />
+  <xacro:SimpleTransmission trans="${prefix}leg2_trans3" joint="${prefix}joint3_2" actuator="${prefix}leg2_motor3" />
+  <!-- Leg 3 Transmissions -->
+  <xacro:SimpleTransmission trans="${prefix}leg3_trans1" joint="${prefix}joint1_3" actuator="${prefix}leg3_motor1" />
+  <xacro:SimpleTransmission trans="${prefix}leg3_trans2" joint="${prefix}joint2_3" actuator="${prefix}leg3_motor2" />
+  <xacro:SimpleTransmission trans="${prefix}leg3_trans3" joint="${prefix}joint3_3" actuator="${prefix}leg3_motor3" />
+  <!-- Leg 4 Transmissions -->
+  <xacro:SimpleTransmission trans="${prefix}leg4_trans1" joint="${prefix}joint1_4" actuator="${prefix}leg4_motor1" />
+  <xacro:SimpleTransmission trans="${prefix}leg4_trans2" joint="${prefix}joint2_4" actuator="${prefix}leg4_motor2" />
+  <xacro:SimpleTransmission trans="${prefix}leg4_trans3" joint="${prefix}joint3_4" actuator="${prefix}leg4_motor3" />
+  <!-- Leg 5 Transmissions -->
+  <xacro:SimpleTransmission trans="${prefix}leg5_trans1" joint="${prefix}joint1_5" actuator="${prefix}leg5_motor1" />
+  <xacro:SimpleTransmission trans="${prefix}leg5_trans2" joint="${prefix}joint2_5" actuator="${prefix}leg5_motor2" />
+  <xacro:SimpleTransmission trans="${prefix}leg5_trans3" joint="${prefix}joint3_5" actuator="${prefix}leg5_motor3" />
+  <!-- Leg 6 Transmissions -->
+  <xacro:SimpleTransmission trans="${prefix}leg6_trans1" joint="${prefix}joint1_6" actuator="${prefix}leg6_motor1" />
+  <xacro:SimpleTransmission trans="${prefix}leg6_trans2" joint="${prefix}joint2_6" actuator="${prefix}leg6_motor2" />
+  <xacro:SimpleTransmission trans="${prefix}leg6_trans3" joint="${prefix}joint3_6" actuator="${prefix}leg6_motor3" />
   </xacro:macro>
 </robot>

File: simulation/ros2_ws_hex/src/hexapod_description/urdf/hexapod_leg_ee.urdf.xacro (robot description, xacro)
@@ -119,5 +119,5 @@
       <parent link="${prefix}link3_1"/>
       <child link="${prefix}link4_1"/>
-      <origin xyz="-0.054636	0.071451	0.00505" rpy="1.4072 0 0"/>
+      <origin xyz="-0.054636	0.071451	0.00505" rpy="0 0 0"/>
       <axis xyz="-0.6074290528 -0.794374 0"/>
       <limit effort="5.0" velocity="1.0" lower="0" upper="1.570796327"/>
@@ -232,5 +232,5 @@
       <parent link="${prefix}link3_2"/>
       <child link="${prefix}link4_2"/>
-      <origin xyz="0.0	0.089946	0.00505" rpy="1.4072 0 0"/>
+      <origin xyz="0.0	0.089946	0.00505" rpy="0 0 0"/>
       <axis xyz="-1 0 0"/>
       <limit effort="5.0" velocity="1.0" lower="0" upper="1.570796327"/>
@@ -345,5 +345,5 @@
       <parent link="${prefix}link3_3"/>
       <child link="${prefix}link4_3"/>
-      <origin xyz="0.054636	0.071451	0.00505" rpy="1.4072 0 0"/>
+      <origin xyz="0.054636	0.071451	0.00505" rpy="0 0 0"/>
       <axis xyz="-0.794374 0.6074290528 0"/>
       <limit effort="5.0" velocity="1.0" lower="0" upper="1.570796327"/>
@@ -458,5 +458,5 @@
       <parent link="${prefix}link3_4"/>
       <child link="${prefix}link4_4"/>
-      <origin xyz="0.054636	-0.071451	0.00505" rpy="1.4072 0 0"/>
+      <origin xyz="0.054636	-0.071451	0.00505" rpy="0 0 0"/>
       <axis xyz="0.6074290528 0.794374 0"/>
       <limit effort="5.0" velocity="1.0" lower="0" upper="1.570796327"/>
@@ -571,5 +571,5 @@
       <parent link="${prefix}link3_5"/>
       <child link="${prefix}link4_5"/>
-      <origin xyz="0.0	-0.089946	0.00505" rpy="1.4072 0 0"/>
+      <origin xyz="0.0	-0.089946	0.00505" rpy="0 0 0"/>
       <axis xyz="1 0 0"/>
       <limit effort="5.0" velocity="1.0" lower="0" upper="1.570796327"/>
@@ -684,5 +684,5 @@
       <parent link="${prefix}link3_6"/>
       <child link="${prefix}link4_6"/>
-      <origin xyz="-0.054636	-0.071451	0.00505" rpy="1.4072 0 0"/>
+      <origin xyz="-0.054636	-0.071451	0.00505" rpy="0 0 0"/>
       <axis xyz="0.794374 -0.6074290528 0"/>
       <limit effort="5.0" velocity="1.0" lower="0" upper="1.570796327"/>
@@ -716,36 +716,4 @@
     </link>
     <!-- END EFFECTOR JOINT AND LINK -->
-<!--may be useful to set leg in starting position
-    <transmission name="${prefix}trans_joint1_6">
-      <type>transmission_interface/SimpleTransmission</type>
-      <joint name="${prefix}joint1_6">
-        <hardwareInterface>hardware_interface/PositionJointInterface</hardwareInterface>
-      </joint>
-      <actuator name="${prefix}motor1_6">
-        <hardwareInterface>hardware_interface/PositionJointInterface</hardwareInterface>
-        <mechanicalReduction>1.0</mechanicalReduction>
-      </actuator>
-    </transmission>
-    <transmission name="${prefix}trans_joint2_6">
-      <type>transmission_interface/SimpleTransmission</type>
-      <joint name="${prefix}joint2_6">
-        <hardwareInterface>hardware_interface/PositionJointInterface</hardwareInterface>
-      </joint>
-      <actuator name="${prefix}motor2_6">
-        <hardwareInterface>hardware_interface/PositionJointInterface</hardwareInterface>
-        <mechanicalReduction>1.0</mechanicalReduction>
-      </actuator>
-    </transmission>
-    <transmission name="${prefix}trans_joint3_6">
-      <type>transmission_interface/SimpleTransmission</type>
-      <joint name="${prefix}joint3_6">
-        <hardwareInterface>hardware_interface/PositionJointInterface</hardwareInterface>
-      </joint>
-      <actuator name="${prefix}motor3_6">
-        <hardwareInterface>hardware_interface/PositionJointInterface</hardwareInterface>
-        <mechanicalReduction>1.0</mechanicalReduction>
-      </actuator>
-    </transmission>
-    -->
     <joint name="${prefix}joint4_6" type="fixed">
       <parent link="${prefix}link4_6"/>
