Commit message: I fixed the incorrect display of the model in gazebo. I removed unnecessary stl files. I added loading by gazebo of ROS2 controllers.

File: simulation/ros2_ws_hex/src/hexapod_description/collision/down_section_hitbox.xacro (robot description, xacro)
@@ -29,5 +29,5 @@
         <xacro:property name="cube_2_offset_z" value="0.0"/>
         <!-- Cylinder 1 - CSV: cylinder_1,"0,425","0,425","0,65","-0,00025391","0,0926495",0,"1,570796327",0,0 -->
-        <xacro:property name="cylinder_1_radius" value="0.00850"/>  <!-- Doubled from 0.00425 -->
+        <xacro:property name="cylinder_1_radius" value="0.00425"/>  <!-- Doubled from 0.00425 -->
         <xacro:property name="cylinder_1_length" value="0.0130"/>   <!-- Doubled from 0.0065 -->
         <xacro:property name="cylinder_1_offset_x" value="-0.00025391"/>
@@ -35,5 +35,5 @@
         <xacro:property name="cylinder_1_offset_z" value="0.0"/>
         <!-- Sphere 1 - CSV: sphere_1,"0,425","0,425","0,425","-0,00025391","0,0992194",0,0,0,0 -->
-        <xacro:property name="sphere_1_radius" value="0.00850"/>  <!-- Doubled from 0.00425 -->
+        <xacro:property name="sphere_1_radius" value="0.00425"/>  <!-- Doubled from 0.00425 -->
         <xacro:property name="sphere_1_offset_x" value="-0.00025391"/>
         <xacro:property name="sphere_1_offset_y" value="0.0992194"/>

File: simulation/ros2_ws_hex/src/hexapod_description/ros2_control/hexapod_system.ros2_control.xacro (robot description, xacro)
@@ -2,6 +2,6 @@
 <!-- DLA SYMULACJI WAŻNE SĄ JEDYNIE LINIJKI 11 - 15 -->
 <robot xmlns:xacro="http://www.ros.org/wiki/xacro">
-  <xacro:macro name="hexapod_system" params="name prefix port_name:=/dev/ttyUSB0 use_sim:=^|false use_fake_hardware:=^|false fake_sensor_commands:=^|false">
-    <ros2_control name="omx" type="system">
+  <xacro:macro name="hexapod_system" params="use_sim prefix">
+    <ros2_control name="hexapod" type="system">
       <xacro:if value="$(arg use_sim)">
         <hardware>
@@ -9,51 +9,4 @@
         </hardware>
       </xacro:if>
-      <xacro:unless value="$(arg use_sim)">
-        <hardware>
-          <xacro:if value="${use_fake_hardware}">
-            <plugin>fake_components/GenericSystem</plugin>
-            <param name="fake_sensor_commands">${fake_sensor_commands}</param>
-            <param name="state_following_offset">0.0</param>
-          </xacro:if>
-          <xacro:unless value="${use_fake_hardware}">
-            <plugin>dynamixel_hardware_interface/DynamixelHardware</plugin>
-            <param name="port_name">${port_name}</param>
-            <param name="baud_rate">1000000</param>
-            <param name="error_timeout_sec">0.2</param>
-            <param name="dynamixel_model_folder">/param/dxl_model</param>
-            <param name="number_of_joints">5</param>
-            <param name="number_of_transmissions">5</param>
-            <param name="transmission_to_joint_matrix">
-              1, 0, 0, 0, 0,
-              0, 1, 0, 0, 0,
-              0, 0, 1, 0, 0,
-              0, 0, 0, 1, 0,
-              0, 0, 0, 0, 1
-            </param>
-            <param name="joint_to_transmission_matrix">
-              1, 0, 0, 0, 0,
-              0, 1, 0, 0, 0,
-              0, 0, 1, 0, 0,
-              0, 0, 0, 1, 0,
-              0, 0, 0, 0, 1
-            </param>
-            <param name="ros_update_freq">200</param>
-            <param name="dynamixel_state_pub_msg_name">dynamixel_hardware_interface/dxl_state</param>
-            <param name="get_dynamixel_data_srv_name">dynamixel_hardware_interface/get_dxl_data</param>
-            <param name="set_dynamixel_data_srv_name">dynamixel_hardware_interface/set_dxl_data</param>
-            <param name="reboot_dxl_srv_name">dynamixel_hardware_interface/reboot_dxl</param>
-            <param name="set_dxl_torque_srv_name">dynamixel_hardware_interface/set_dxl_torque</param>
-              <!-- This parameter is used for a prismatic joint
-            that operates through a revolute mechanism. If the joint does not require this configuration, this parameter can be removed. -->
-            <param name="use_revolute_to_prismatic_gripper">1</param>
-            <param name="revolute_to_prismatic_dxl">dxl5</param>
-            <param name="revolute_max">-1.52</param>
-            <param name="revolute_min">0.92</param>
-            <param name="revolute_to_prismatic_joint">${prefix}gripper_left_joint</param>
-            <param name="prismatic_max">0.019</param>
-            <param name="prismatic_min">-0.01</param>
-          </xacro:unless>
-        </hardware>
-      </xacro:unless>
       <!-- LEG 1 -->
       <joint name="${prefix}joint1_1">
@@ -170,78 +123,4 @@
         <state_interface name="effort"/>
       </joint>
-      <gpio name="dxl1">
-        <param name="type">dxl</param>
-        <param name="ID">11</param>
-        <command_interface name="Goal Position"/>
-        <state_interface name="Present Position"/>
-        <state_interface name="Present Velocity"/>
-        <state_interface name="Present Current"/>
-        <state_interface name="Torque Enable"/>
-        <state_interface name="Present Input Voltage"/>
-        <param name="Position P Gain">800</param>
-        <param name="Position I Gain">100</param>
-        <param name="Position D Gain">100</param>
-        <param name="Profile Velocity">200</param>
-        <param name="Profile Acceleration">50</param>
-        <param name="Drive Mode">0</param>
-      </gpio>
-      <gpio name="dxl2">
-        <param name="type">dxl</param>
-        <param name="ID">12</param>
-        <command_interface name="Goal Position"/>
-        <state_interface name="Present Position"/>
-        <state_interface name="Present Velocity"/>
-        <state_interface name="Present Current"/>
-        <state_interface name="Torque Enable"/>
-        <state_interface name="Present Input Voltage"/>
-        <param name="Position P Gain">800</param>
-        <param name="Position I Gain">100</param>
-        <param name="Position D Gain">100</param>
-        <param name="Profile Velocity">200</param>
-        <param name="Profile Acceleration">50</param>
-        <param name="Drive Mode">0</param>
-      </gpio>
-      <gpio name="dxl3">
-        <param name="type">dxl</param>
-        <param name="ID">13</param>
-        <command_interface name="Goal Position"/>
-        <state_interface name="Present Position"/>
-        <state_interface name="Present Velocity"/>
-        <state_interface name="Present Current"/>
-        <state_interface name="Torque Enable"/>
-        <state_interface name="Present Input Voltage"/>
-        <param name="Position P Gain">800</param>
-        <param name="Position I Gain">100</param>
-        <param name="Position D Gain">100</param>
-        <param name="Profile Velocity">200</param>
-        <param name="Profile Acceleration">50</param>
-        <param name="Drive Mode">0</param>
-      </gpio>
-      <gpio name="dxl4">
-        <param name="type">dxl</param>
-        <param name="ID">14</param>
-        <command_interface name="Goal Position"/>
-        <state_interface name="Present Position"/>
-        <state_interface name="Present Velocity"/>
-        <state_interface name="Present Current"/>
-        <state_interface name="Torque Enable"/>
-        <state_interface name="Present Input Voltage"/>
-        <param name="Position P Gain">800</param>
-        <param name="Position I Gain">100</param>
-        <param name="Position D Gain">100</param>
-        <param name="Profile Velocity">200</param>
-        <param name="Profile Acceleration">50</param>
-        <param name="Drive Mode">0</param>
-      </gpio>
-      <gpio name="dxl5">
-        <param name="type">dxl</param>
-        <param name="ID">15</param>
-        <command_interface name="Goal Position"/>
-        <state_interface name="Present Position"/>
-        <state_interface name="Present Velocity"/>
-        <state_interface name="Present Current"/>
-        <state_interface name="Torque Enable"/>
-        <state_interface name="Present Input Voltage"/>
-      </gpio>
     </ros2_control>
   </xacro:macro>

File: simulation/ros2_ws_hex/src/hexapod_description/urdf/hexapod_ee.urdf.xacro (robot description, xacro)
@@ -1,26 +1,17 @@
 <?xml version="1.0"?>
-<!-- OpenManipulator Chain -->
 <robot name="hexapod" xmlns:xacro="http://ros.org/wiki/xacro">
+  <xacro:arg name="use_sim" default="true" />
   <xacro:arg name="prefix" default="" />
-  <!-- <xacro:arg name="use_sim" default="false" /> -->
-  <!-- <xacro:arg name="use_fake_hardware" default="true" /> -->
-  <!-- <xacro:arg name="fake_sensor_commands" default="false" /> -->
-  <!-- <xacro:arg name="port_name" default="/dev/ttyUSB0" /> -->
-  <!-- Import all Gazebo-customization elements, including Gazebo colors -->
-  <!-- <xacro:include filename="$(find hexapod_description)/gazebo/hexapod.gazebo.xacro" /> -->
-  <!-- Import URDF -->
+  <xacro:include filename="$(find hexapod_description)/gazebo/hexapod.gazebo.xacro" />
   <xacro:include filename="$(find hexapod_description)/urdf/hexapod_leg_ee.urdf.xacro" />
-  <!-- <xacro:include filename="$(find hexapod_description)/ros2_control/hexapod_system.ros2_control.xacro" /> -->
+  <xacro:include filename="$(find hexapod_description)/urdf/hexapod_gazebo.urdf.xacro" />
+  <xacro:include filename="$(find hexapod_description)/ros2_control/hexapod_system.ros2_control.xacro" />
   <xacro:hexapod prefix="$(arg prefix)" />
-  <!-- <xacro:hexapod_gazebo prefix="$(arg prefix)" />
-  <xacro:hexapod_system
-    name="HexapodSystem" prefix="$(arg prefix)" use_sim="$(arg use_sim)"
-    use_fake_hardware="$(arg use_fake_hardware)"
-    fake_sensor_commands="$(arg fake_sensor_commands)"
-    port_name="$(arg port_name)"/> -->
-  <!-- <gazebo>
+  <xacro:hexapod_gazebo prefix="$(arg prefix)" />
+  <xacro:hexapod_system use_sim="$(arg use_sim)" prefix="$(arg prefix)"/>
+  <gazebo>
     <plugin filename="gz_ros2_control-system" name="gz_ros2_control::GazeboSimROS2ControlPlugin">
       <parameters>$(find hex_gz)/config/gazebo_controller_manager.yaml</parameters>
     </plugin>
-  </gazebo> -->
+  </gazebo>
 </robot>

File: simulation/ros2_ws_hex/src/hexapod_description/urdf/hexapod_leg_ee.urdf.xacro (robot description, xacro)
@@ -10,8 +10,8 @@
        value="package://hexapod_description/meshes"/>
    <!-- Include macro modeli kolizyjnych z prostych kształtów geometrycznych -->
-   <xacro:include filename="$(find hexapod_description)/meshes/platform_hitbox.xacro"/>
-   <xacro:include filename="$(find hexapod_description)/meshes/up_section_hitbox.xacro"/>
-   <xacro:include filename="$(find hexapod_description)/meshes/mid_section_hitbox.xacro"/>
-   <xacro:include filename="$(find hexapod_description)/meshes/down_section_hitbox.xacro"/>
+   <xacro:include filename="$(find hexapod_description)/collision/platform_hitbox.xacro"/>
+   <xacro:include filename="$(find hexapod_description)/collision/up_section_hitbox.xacro"/>
+   <xacro:include filename="$(find hexapod_description)/collision/mid_section_hitbox.xacro"/>
+   <xacro:include filename="$(find hexapod_description)/collision/down_section_hitbox.xacro"/>
    <!-- Macro platformy -->
     <xacro:macro name="platform_base" params="prefix">
