Commit message: I added new robot model to the simulation and optimized simulation for both models. New model on default. Old model gazebov1.launch.py

File: sim_and_real/ros2_ws_hex/src/hexapod_description/urdf/imu.urdf.xacro (robot description, xacro)
@@ -2,4 +2,5 @@
 <robot xmlns:xacro="http://www.ros.org/wiki/xacro">
     <xacro:property name="M_PI" value="3.1415926535897931" />
+    <xacro:arg name="prefix" default=""/>
     <!-- imu jest ale nie wysyla nic -> do naprawy :( -->
     <xacro:macro name="imu_sensor" params="

File: sim_and_real/ros2_ws_hex/src/hexapod_moveit_config/config/hexapod.urdf.xacro (robot description, xacro)
@@ -3,4 +3,4 @@
     <xacro:arg name="use_gazebo" default="false" />
     <xacro:include filename="$(find hexapod_description)/urdf/hexapod_ee.urdf.xacro" />
-    <xacro:hexapod_ee use_sim="true" prefix="" use_gazebo="$(arg use_gazebo)"/>
+    <xacro:hexapod_ee use_sim="true" prefix="" use_gazebo="$(arg use_gazebo)" version="2"/>
 </robot>

Commit message: Started implementing proper hardware interface. Fake hardware is working

File: sim_and_real/ros2_ws_hex/src/hexapod_description/urdf/hexapod.urdf.xacro (robot description, xacro)
@@ -1,11 +1,20 @@
 <?xml version="1.0"?>
 <robot name="hexapod" xmlns:xacro="http://ros.org/wiki/xacro">
-    <!-- Declare the argument with a default value -->
-    <xacro:arg name="use_gazebo" default="true"/>
-    <xacro:arg name="version" default="2"/>
-    <xacro:property name="use_gazebo" value="$(arg use_gazebo)"/>
-    <xacro:property name="version" value="$(arg version)"/>
+    <xacro:arg name="prefix" default="" />
+    <xacro:arg name="use_gazebo" default="false" />
+    <xacro:arg name="use_fake_hardware" default="false" />
+    <xacro:arg name="fake_sensor_commands" default="false" />
+    <xacro:arg name="port_name" default="/dev/ttyUSB0" />
+    <xacro:arg name="baud_rate" default="115200" />
+    <xacro:arg name="version" default="2" />
     <xacro:include filename="$(find hexapod_description)/urdf/hexapod_ee.urdf.xacro" />
-    <!-- Pass the argument value to the macro -->
-    <xacro:hexapod_ee use_sim="true" prefix="" use_gazebo="$(arg use_gazebo)" version="$(arg version)"/>
+    <xacro:hexapod_ee
+        use_sim="true"
+        prefix="$(arg prefix)"
+        use_gazebo="$(arg use_gazebo)"
+        use_fake_hardware="$(arg use_fake_hardware)"
+        fake_sensor_commands="$(arg fake_sensor_commands)"
+        port_name="$(arg port_name)"
+        baud_rate="$(arg baud_rate)"
+        version="$(arg version)" />
 </robot>

File: sim_and_real/ros2_ws_hex/src/hexapod_description/urdf/hexapod_ee.urdf.xacro (robot description, xacro)
@@ -1,5 +1,5 @@
 <?xml version="1.0"?>
 <robot name="hexapod" xmlns:xacro="http://ros.org/wiki/xacro">
-  <xacro:macro name="hexapod_ee" params="use_sim prefix use_gazebo version">
+  <xacro:macro name="hexapod_ee" params="use_sim prefix use_gazebo use_fake_hardware fake_sensor_commands port_name baud_rate version">
     <xacro:include filename="$(find hexapod_description)/gazebo/hexapod.gazebo.xacro" />
     <xacro:include filename="$(find hexapod_description)/urdf/hexapod_leg_ee.urdf.xacro" />
@@ -38,5 +38,12 @@
     <!-- <xacro:hexapod_ros2_control name="FakeSystem" initial_positions_file="$(arg initial_positions_file)"/> -->
     <!-- <xacro:hexapod_ros2_control use_sim="$(arg use_sim)" prefix="$(arg prefix)" initial_positions_file="$(find hexapod_description)/config/initial_positions.yaml"/>  -->
-    <xacro:hexapod_ros2_control name="hexapod" initial_positions_file="$(find hexapod_description)/config/initial_positions.yaml" use_gazebo="${use_gazebo}"/>
+    <xacro:hexapod_ros2_control
+        name="hexapod"
+        initial_positions_file="$(find hexapod_description)/config/initial_positions.yaml"
+        use_gazebo="${use_gazebo}"
+        use_fake_hardware="${use_fake_hardware}"
+        fake_sensor_commands="${fake_sensor_commands}"
+        port_name="${port_name}"
+        baud_rate="${baud_rate}" />
   </xacro:macro>
 </robot>

File: sim_and_real/ros2_ws_hex/src/hexapod_moveit_config/config/hexapod.ros2_control.xacro (robot description, xacro)
@@ -1,20 +1,32 @@
 <?xml version="1.0"?>
 <robot xmlns:xacro="http://www.ros.org/wiki/xacro">
-    <xacro:macro name="hexapod_ros2_control" params="name initial_positions_file use_gazebo">
+    <xacro:macro name="hexapod_ros2_control" params="name initial_positions_file use_gazebo use_fake_hardware:=false fake_sensor_commands port_name baud_rate">
         <xacro:property name="initial_positions" value="${xacro.load_yaml(initial_positions_file)['initial_positions']}"/>
         <ros2_control name="${name}" type="system">
+        <!-- Gazebo simulation (priorytet 1) -->
         <xacro:if value="${use_gazebo}">
             <hardware>
-                <!-- By default, set up controllers for simulation. This won't work on real hardware -->
                 <plugin>gz_ros2_control/GazeboSimSystem</plugin>
-                <!-- <plugin>mock_components/GenericSystem</plugin> -->
             </hardware>
         </xacro:if>
+        <!-- Fake hardware for testing (priorytet 2) -->
         <xacro:unless value="${use_gazebo}">
-            <hardware>
-                <!-- By default, set up controllers for simulation. This won't work on real hardware -->
-                <!-- <plugin>gz_ros2_control/GazeboSimSystem</plugin> -->
-                <plugin>mock_components/GenericSystem</plugin>
-            </hardware>
+            <xacro:if value="${use_fake_hardware}">
+                <hardware>
+                    <plugin>mock_components/GenericSystem</plugin>
+                    <param name="fake_sensor_commands">${fake_sensor_commands}</param>
+                    <param name="state_following_offset">0.0</param>
+                </hardware>
+            </xacro:if>
+        </xacro:unless>
+        <!-- Real hardware with ESP32 (priorytet 3) -->
+        <xacro:unless value="${use_gazebo}">
+            <xacro:unless value="${use_fake_hardware}">
+                <hardware>
+                    <plugin>hexapod_hardware/HexapodHardwareInterface</plugin>
+                    <param name="port_name">${port_name}</param>
+                    <param name="baud_rate">${baud_rate}</param>
+                </hardware>
+            </xacro:unless>
         </xacro:unless>
             <!-- Leg 1 joints -->

File: sim_and_real/ros2_ws_hex/src/hexapod_moveit_config/config/hexapod.urdf.xacro (robot description, xacro)
@@ -1,6 +1,20 @@
 <?xml version="1.0"?>
 <robot name="hexapod" xmlns:xacro="http://ros.org/wiki/xacro">
+    <xacro:arg name="prefix" default="" />
     <xacro:arg name="use_gazebo" default="false" />
+    <xacro:arg name="use_fake_hardware" default="false" />
+    <xacro:arg name="fake_sensor_commands" default="false" />
+    <xacro:arg name="port_name" default="/dev/ttyUSB0" />
+    <xacro:arg name="baud_rate" default="115200" />
+    <xacro:arg name="version" default="2" />
     <xacro:include filename="$(find hexapod_description)/urdf/hexapod_ee.urdf.xacro" />
-    <xacro:hexapod_ee use_sim="true" prefix="" use_gazebo="$(arg use_gazebo)" version="2"/>
+    <xacro:hexapod_ee
+        use_sim="true"
+        prefix="$(arg prefix)"
+        use_gazebo="$(arg use_gazebo)"
+        use_fake_hardware="$(arg use_fake_hardware)"
+        fake_sensor_commands="$(arg fake_sensor_commands)"
+        port_name="$(arg port_name)"
+        baud_rate="$(arg baud_rate)"
+        version="$(arg version)" />
 </robot>
